File: WirelessEStop_Tx/WirelessEStop_Tx.sch (KiCad schematic (older format))
At the start: 14 parts

Commit message: Fixed files and stuff
Organized some files and also worked on the footprint assignments and started to create a footprint for one of the three switches.
Parts:
- removed C? (x2): CP1_Small, symbol Device:CP1_Small
- added C1, C2: 10u, Capacitor_SMD:C_0603_1608Metric_Pad1.05x0.95mm_HandSolder, symbol Device:C_Small
- Conn1: renamed from Conn?; footprint (none) -> MRDT_Connectors:MOLEX_SL_02_Horizontal
- D1: renamed from D?; value D_Schottky -> 3.3V_Schottky; footprint (none) -> Diode_SMD:D_0603_1608Metric_Pad1.05x0.95mm_HandSolder
- D2: renamed from D?; footprint (none) -> LED_SMD:LED_0603_1608Metric_Pad1.05x0.95mm_HandSolder
- L1: renamed from L?; footprint (none) -> Inductor_SMD:L_0603_1608Metric_Pad1.05x0.95mm_HandSolder
- R1, R2, R3: renamed from R?; footprint (none) -> Resistor_SMD:R_0603_1608Metric_Pad1.05x0.95mm_HandSolder
- U2: renamed from U?; footprint (none) -> Package_SO:SOIC-8_3.9x4.9mm_P1.27mm
- gave numbers to parts that had none: 4
Connections:
- wire segments 47 -> 48

Commit message: More footprint updates
Made a footprint for the ESP8266-01, but it still needs to be checked.
Parts:
- SW1: footprint (none) -> WirelessEStop:MOMSwitch_SPDT
- SW2: footprint (none) -> WirelessEStop:ToggleSwitch_SPDT
- SW3: footprint (none) -> WirelessEStop:SlideSwitch_SPDT
- U1: footprint (none) -> WirelessEStop:ESP8266-01
Changed lines of the file:
@@
 F 0 "SW3" H 6750 3085 50  0000 C CNN
 F 1 "Master Power" H 6750 2994 50  0000 C CNN
-F 2 "" H 6750 2850 50  0001 C CNN
+F 2 "WirelessEStop:SlideSwitch_SPDT" H 6750 2850 50  0001 C CNN
 F 3 "" H 6750 2850 50  0001 C CNN
 	1    6750 2850
@@
 F 0 "SW2" H 3950 5100 50  0000 C CNN
 F 1 "Maintain Switch" H 3950 5200 50  0000 C CNN
-F 2 "" H 3900 5300 50  0001 C CNN
+F 2 "WirelessEStop:ToggleSwitch_SPDT" H 3900 5300 50  0001 C CNN
 F 3 "" H 3900 5300 50  0001 C CNN
 	1    3900 5300
@@
 F 0 "SW1" H 3150 4750 50  0000 C CNN
 F 1 "MOM Switch" H 3150 4650 50  0000 C CNN
-F 2 "" H 3050 4700 50  0001 C CNN
+F 2 "WirelessEStop:MOMSwitch_SPDT" H 3050 4700 50  0001 C CNN
 F 3 "" H 3050 4700 50  0001 C CNN
 	1    3050 4500
@@
 F 0 "U1" H 4650 4575 50  0000 C CNN
 F 1 "ESP_8266_01" H 4650 4484 50  0000 C CNN
-F 2 "" H 4600 4450 50  0001 C CNN
+F 2 "WirelessEStop:ESP8266-01" H 4600 4450 50  0001 C CNN
 F 3 "" H 4600 4450 50  0001 C CNN
 	1    4650 4350

Commit message: 1st Board Review Changes
Made a little bit of progress on some of the changes that needed to be made after the board review.
Parts:
- removed SW2: Maintain Switch, WirelessEStop:ToggleSwitch_SPDT, symbol Switch:SW_SPST
- added D3, D4, D5, D?: LED, LED_SMD:LED_0603_1608Metric_Pad1.05x0.95mm_HandSolder, symbol Device:LED
- added R4, R5, R6, R?: 500, Resistor_SMD:R_0603_1608Metric_Pad1.05x0.95mm_HandSolder, symbol Device:R
- added SW2: Maintain Switch, WirelessEStop:ToggleSwitch_SPDT, symbol Switch:SW_SPDT_MSM
- R3: value 150 -> 500
- SW1: footprint WirelessEStop:MOMSwitch_SPDT -> WirelessEStop:D6_SPST
Connections:
- net labels added: +3.3V, D1, MOM_IN, Maintain_IN
- net labels removed: +3V3
- wire segments 48 -> 64

Commit message: Finished up the Transmitter Schematic
Just more work done
Parts:
- gave numbers to parts that had none: 2
- renumbered D1 to D0
Connections:
- net labels added: SW_EStop, SW_Link_EN
- net labels removed: D1
- wire segments 64 -> 75
- no-connect marks 0 -> 1
Other:
- note added: "Blue"
- note added: "D1"
- note added: "Green"
- note added: "LEDs"
- note added: "Red"
- note added: "Yellow"

Commit message: Revert "Finished up the Transmitter Schematic"
This reverts commit 0529c396fdec7017beb922822e4a7a479dabca41.
Parts:
- renumbered D0 to D1, D1 to D?, R7 to R?
Connections:
- net labels added: D1
- net labels removed: SW_EStop, SW_Link_EN
- wire segments 75 -> 64
- no-connect marks 1 -> 0
Other:
- note removed: "Blue"
- note removed: "D1"
- note removed: "Green"
- note removed: "LEDs"
- note removed: "Red"
- note removed: "Yellow"
