File: WirelessEStop_Tx/WirelessEStop_Tx.sch (KiCad schematic (older format))
At the start: 22 parts, among them SW1 MOM Switch, SW2 Maintain Switch, SW3 Master Power, U1 ESP_8266_01, U2 AP1059

Commit message: Worked on Board Layout
Pretty much finished the board. Need the BOM and stuff yet.
Parts:
- SW3: footprint WirelessEStop:SlideSwitch_SPDT -> WirelessEStop:SlideSwitch_SPST
Changed lines of the file:
@@
 F 0 "SW3" H 5900 2785 50  0000 C CNN
 F 1 "Master Power" H 5900 2694 50  0000 C CNN
-F 2 "WirelessEStop:SlideSwitch_SPDT" H 5900 2550 50  0001 C CNN
+F 2 "WirelessEStop:SlideSwitch_SPST" H 5900 2550 50  0001 C CNN
 F 3 "" H 5900 2550 50  0001 C CNN
 	1    5900 2550

Commit message: Updated Schematic
Changed AP1509 back to an OKI
Parts:
- removed D0: 3.3V_Schottky, Diode_SMD:D_0603_1608Metric_Pad1.05x0.95mm_HandSolder, symbol Device:D_Schottky
- removed L1: 47uH Inductor, Inductor_SMD:L_0603_1608Metric_Pad1.05x0.95mm_HandSolder, symbol pspice:INDUCTOR
- removed U2: AP1059, Package_SO:SOIC-8_3.9x4.9mm_P1.27mm, symbol MRDT_ICs:AP1059
- added U?: OKI, symbol MRDT_Devices:OKI
Connections:
- wire segments 75 -> 51
Changed lines of the file:
@@
 L MRDT_Connectors:Molex_SL_02 Conn1
 U 1 1 5BD1365E
-P 6500 2500
-F 0 "Conn1" H 6800 2550 60  0000 C CNN
-F 1 "9V Batt" H 6800 2650 60  0000 C CNN
-F 2 "MRDT_Connectors:MOLEX_SL_02_Horizontal" H 6500 2400 60  0001 C CNN
-F 3 "" H 6500 2400 60  0001 C CNN
-	1    6500 2500
+P 6050 2900
+F 0 "Conn1" H 6350 2950 60  0000 C CNN
+F 1 "9V Batt" H 6350 3050 60  0000 C CNN
+F 2 "MRDT_Connectors:MOLEX_SL_02_Horizontal" H 6050 2800 60  0001 C CNN
+F 3 "" H 6050 2800 60  0001 C CNN
+	1    6050 2900
 	1    0    0    1
 $EndComp
@@
 L Switch:SW_SPST SW3
 U 1 1 5BD233CE
-P 5900 2550
-F 0 "SW3" H 5900 2785 50  0000 C CNN
-F 1 "Master Power" H 5900 2694 50  0000 C CNN
-F 2 "WirelessEStop:SlideSwitch_SPST" H 5900 2550 50  0001 C CNN
-F 3 "" H 5900 2550 50  0001 C CNN
-	1    5900 2550
+P 5450 2950
+F 0 "SW3" H 5450 3185 50  0000 C CNN
+F 1 "Master Power" H 5450 3094 50  0000 C CNN
+F 2 "WirelessEStop:SlideSwitch_SPST" H 5450 2950 50  0001 C CNN
+F 3 "" H 5450 2950 50  0001 C CNN
+	1    5450 2950
 	1    0    0    -1
 $EndComp
@@
 $EndComp
 Wire Wire Line
-	6300 2550 6100 2550
-Text Label 6250 2550 2    50   ~ 0
+	5850 2950 5650 2950
+Text Label 5800 2950 2    50   ~ 0
 Vin
 $Comp
@@
 F 3 "" H 3450 4550 50  0001 C CNN
 	1    3450 4550
-	1    0    0    -1
-$EndComp
-$Comp
-L power:GND #PWR0102
-U 1 1 5BD242B2
-P 6250 2700
-F 0 "#PWR0102" H 6250 2450 50  0001 C CNN
-F 1 "GND" H 6255 2527 50  0000 C CNN
-F 2 "" H 6250 2700 50  0001 C CNN
-F 3 "" H 6250 2700 50  0001 C CNN
-	1    6250 2700
 	1    0    0    -1
 $EndComp
@@
 	2950 5000 2950 5050
 $Comp
-L MRDT_ICs:AP1059 U2
-U 1 1 5BDE1FD8
-P 4450 2200
-F 0 "U2" H 4700 2750 60  0000 C CNN
-F 1 "AP1059" H 4700 2650 60  0000 C CNN
-F 2 "Package_SO:SOIC-8_3.9x4.9mm_P1.27mm" H 4200 2100 60  0001 C CNN
-F 3 "" H 4200 2100 60  0001 C CNN
-	1    4450 2200
-	-1   0    0    1
-$EndComp
-$Comp
 L power:GND #PWR0109
 U 1 1 5BDE49F4
-P 3450 2550
-F 0 "#PWR0109" H 3450 2300 50  0001 C CNN
-F 1 "GND" H 3455 2377 50  0000 C CNN
-F 2 "" H 3450 2550 50  0001 C CNN
-F 3 "" H 3450 2550 50  0001 C CNN
-	1    3450 2550
-	1    0    0    -1
-$EndComp
-Wire Wire Line
-	4650 2250 4650 1950
-Wire Wire Line
-	4650 1950 5450 1950
-Wire Wire Line
-	5450 1950 5450 2250
-Wire Wire Line
-	4650 1950 3600 1950
-Connection ~ 4650 1950
-$Comp
-L Device:D_Schottky D0
-U 1 1 5BDE6225
-P 4150 2850
-F 0 "D0" H 4150 3066 50  0000 C CNN
-F 1 "3.3V_Schottky" H 4150 2975 50  0000 C CNN
-F 2 "Diode_SMD:D_0603_1608Metric_Pad1.05x0.95mm_HandSolder" H 4150 2850 50  0001 C CNN
-F 3 "~" H 4150 2850 50  0001 C CNN
-	1    4150 2850
-	-1   0    0    1
-$EndComp
-Wire Wire Line
-	5700 2550 5450 2550
-Wire Wire Line
-	5450 2450 5450 2550
-Connection ~ 5450 2550
-Wire Wire Line
-	5450 2550 4650 2550
-Wire Wire Line
-	4100 3550 3600 3550
-$Comp
-L pspice:INDUCTOR L1
-U 1 1 5BDE91B6
-P 4500 3200
-F 0 "L1" V 4454 3277 50  0000 L CNN
-F 1 "47uH Inductor" V 4545 3277 50  0000 L CNN
-F 2 "Inductor_SMD:L_0603_1608Metric_Pad1.05x0.95mm_HandSolder" H 4500 3200 50  0001 C CNN
-F 3 "" H 4500 3200 50  0001 C CNN
-	1    4500 3200
-	0    1    1    0
-$EndComp
-Wire Wire Line
-	4500 2950 4500 2850
-Wire Wire Line
-	4300 3550 4500 3550
-Wire Wire Line
-	4500 3550 4500 3450
-Connection ~ 4500 3550
-Wire Wire Line
-	4500 3550 5050 3550
-Wire Wire Line
-	5050 2350 4650 2350
-Wire Wire Line
-	5050 3550 5050 2350
-Wire Wire Line
-	4650 2450 4800 2450
-Wire Wire Line
-	4800 2450 4800 2850
-Wire Wire Line
-	4800 2850 4500 2850
-Connection ~ 4500 2850
-Wire Wire Line
-	4500 3550 4500 4050
-Wire Wire Line
-	3600 1950 3600 2550
-Wire Wire Line
-	3800 2250 3750 2250
-Wire Wire Line
-	3750 2250 3750 2350
-Wire Wire Line
-	3750 2550 3800 2550
-Wire Wire Line
-	3800 2450 3750 2450
-Connection ~ 3750 2450
-Wire Wire Line
-	3750 2450 3750 2550
-Wire Wire Line
-	3800 2350 3750 2350
-Connection ~ 3750 2350
-Wire Wire Line
-	3750 2350 3750 2450
-Connection ~ 3750 2550
-Wire Wire Line
-	3450 2550 3600 2550
-Connection ~ 3600 2550
-Wire Wire Line
-	3600 2550 3750 2550
+P 4350 3350
+F 0 "#PWR0109" H 4350 3100 50  0001 C CNN
+F 1 "GND" H 4355 3177 50  0000 C CNN
+F 2 "" H 4350 3350 50  0001 C CNN
+F 3 "" H 4350 3350 50  0001 C CNN
+	1    4350 3350
+	1    0    0    -1
+$EndComp
 Wire Wire Line
 	2000 4200 2000 4150
@@
 L Device:C_Small C1
 U 1 1 5BEC1EDB
-P 4200 3550
-F 0 "C1" V 3971 3550 50  0000 C CNN
-F 1 "10u" V 4062 3550 50  0000 C CNN
-F 2 "Capacitor_SMD:C_0603_1608Metric_Pad1.05x0.95mm_HandSolder" H 4200 3550 50  0001 C CNN
-F 3 "~" H 4200 3550 50  0001 C CNN
-	1    4200 3550
-	0    1    1    0
+P 4950 3150
+F 0 "C1" H 4800 3200 50  0000 C CNN
+F 1 "10u" H 4812 3150 50  0000 C CNN
+F 2 "Capacitor_SMD:C_0603_1608Metric_Pad1.05x0.95mm_HandSolder" H 4950 3150 50  0001 C CNN
+F 3 "~" H 4950 3150 50  0001 C CNN
+	1    4950 3150
+	-1   0    0    1
 $EndComp
 $Comp
 L Device:C_Small C2
 U 1 1 5BEC1F55
-P 5450 2350
-F 0 "C2" H 5200 2400 50  0000 L CNN
-F 1 "10u" H 5200 2300 50  0000 L CNN
-F 2 "Capacitor_SMD:C_0603_1608Metric_Pad1.05x0.95mm_HandSolder" H 5450 2350 50  0001 C CNN
-F 3 "~" H 5450 2350 50  0001 C CNN
-	1    5450 2350
-	1    0    0    -1
+P 3800 3150
+F 0 "C2" H 3900 3200 50  0000 L CNN
+F 1 "10u" H 3900 3100 50  0000 L CNN
+F 2 "Capacitor_SMD:C_0603_1608Metric_Pad1.05x0.95mm_HandSolder" H 3800 3150 50  0001 C CNN
+F 3 "~" H 3800 3150 50  0001 C CNN
+	1    3800 3150
+	-1   0    0    1
 $EndComp
 Wire Wire Line
@@
 	2550 2050 2550 2200
 Wire Wire Line
-	6300 2650 6250 2650
-Wire Wire Line
-	6250 2650 6250 2700
+	5850 3050 5800 3050
 $Comp
 L power:+3.3V #PWR0110
@@
 Wire Wire Line
 	4100 4050 4350 4050
-Connection ~ 4350 4050
-Wire Wire Line
-	4350 4050 4500 4050
 $Comp
 L power:+3.3V #PWR0113
@@
 SW_Link_EN
 Wire Wire Line
-	3600 2550 3600 2850
-Wire Wire Line
-	4300 2850 4500 2850
-Wire Wire Line
-	4000 2850 3600 2850
-Connection ~ 3600 2850
-Wire Wire Line
-	3600 2850 3600 3550
-Wire Wire Line
 	2950 4350 3200 4350
 Connection ~ 2700 4200
@@
 Wire Wire Line
 	2950 4350 2950 5000
+$Comp
+L MRDT_Devices:OKI U?
+U 1 1 5C1A2622
+P 4550 3050
+F 0 "U?" H 4600 3000 60  0001 C CNN
+F 1 "OKI" H 4750 3331 60  0000 C CNN
+F 2 "" H 4350 2950 60  0001 C CNN
+F 3 "" H 4350 2950 60  0001 C CNN
+	1    4550 3050
+	-1   0    0    -1
+$EndComp
+Wire Wire Line
+	4750 2950 4950 2950
+Wire Wire Line
+	5800 3250 4950 3250
+Wire Wire Line
+	5800 3050 5800 3250
+Connection ~ 4350 3250
+Wire Wire Line
+	4350 3250 3800 3250
+Connection ~ 4950 3250
+Wire Wire Line
+	4950 3250 4350 3250
+Wire Wire Line
+	4350 3350 4350 3250
+Wire Wire Line
+	3800 3050 3800 2950
+Wire Wire Line
+	3800 2950 3950 2950
+Wire Wire Line
+	4950 3050 4950 2950
+Connection ~ 4950 2950
+Wire Wire Line
+	4950 2950 5250 2950
+$Comp
+L power:+3.3V #PWR?
+U 1 1 5C1ABFA8
+P 3800 2950
+F 0 "#PWR?" H 3800 2800 50  0001 C CNN
+F 1 "+3.3V" H 3815 3123 50  0000 C CNN
+F 2 "" H 3800 2950 50  0001 C CNN
+F 3 "" H 3800 2950 50  0001 C CNN
+	1    3800 2950
+	1    0    0    -1
+$EndComp
+Connection ~ 3800 2950
 $EndSCHEMATC
