File: WirelessEStop_Tx/WirelessEStop_Tx.sch (KiCad schematic (older format))
At the start: 20 parts, among them SW1 MOM Switch, SW2 Maintain Switch, SW3 Master Power, U1 ESP_8266_01

Commit message: Fixed Board
Changed AP1509 and fixed the ESP8266-01
Parts:
- U2: renamed from U?; footprint (none) -> MRDT_Devices:OKI_Horizontal
Changed lines of the file:
@@
 	2950 4350 2950 5000
 $Comp
-L MRDT_Devices:OKI U?
+L MRDT_Devices:OKI U2
 U 1 1 5C1A2622
 P 4550 3050
-F 0 "U?" H 4600 3000 60  0001 C CNN
+F 0 "U2" H 4600 3000 60  0001 C CNN
 F 1 "OKI" H 4750 3331 60  0000 C CNN
-F 2 "" H 4350 2950 60  0001 C CNN
+F 2 "MRDT_Devices:OKI_Horizontal" H 4350 2950 60  0001 C CNN
 F 3 "" H 4350 2950 60  0001 C CNN
 	1    4550 3050
@@
 	4950 2950 5250 2950
 $Comp
-L power:+3.3V #PWR?
+L power:+3.3V #PWR0102
 U 1 1 5C1ABFA8
 P 3800 2950
-F 0 "#PWR?" H 3800 2800 50  0001 C CNN
+F 0 "#PWR0102" H 3800 2800 50  0001 C CNN
 F 1 "+3.3V" H 3815 3123 50  0000 C CNN
 F 2 "" H 3800 2950 50  0001 C CNN

Commit message: Fixed Errors and made neater
Parts:
- SW2: symbol Switch:SW_SPDT_MSM -> Switch:SW_SPDT
Connections:
- wire segments 51 -> 52
- no-connect marks 1 -> 2
Other:
- note added: "ESP & Switches"
- note added: "POWER"
