File: WirelessEStop_Rx/WirelessEStop_Rx.sch (KiCad schematic (older format))
At the start: 2 parts

Commit message: Made the Reciever Schematic
Parts:
- added C? (x2): C_Small, symbol Device:C_Small
- added Conn? (x2): Molex_SL_02, symbol MRDT_Connectors:Molex_SL_02
- added D? (x2): LED, symbol Device:LED
- added Q?: 2N7002, Package_TO_SOT_SMD:SOT-23, symbol Transistor_FET:2N7002
- added R?: R, symbol Device:R
- added SW?: SW_SPST, symbol Switch:SW_SPST
- added U?: OKI, symbol MRDT_Devices:OKI
Connections:
- wire segments 3 -> 29
