File: WirelessEStop_Rx/WirelessEStop_Rx.sch (KiCad schematic (older format))
At the start: 14 parts, among them Q1 2N7002, U1 OKI, U2 ESP_8266_01

Commit message: Adjusted things & made Gerbs
Other:
- note added: "ESP-01 & E-Stop Circuit"
- note added: "POWER INPUT"
- moved on the sheet: Q1
