File: WirelessEStop_Rx/WirelessEStop_Rx.kicad_pcb (KiCad board)
At the start: 2 copper layers, 53.3 x 30.5 mm, 16 parts, among them Q1 2N7002, U1 OKI, U2 ESP_8266_01

Commit message: Went over a few things
Parts:
- moved G*** 1.30 mm to (149.9, 95.5)
Other:
- board text added: "Off"
- board text added: "On"
Changed lines of the file:
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@@
   (general
     (thickness 1.6)
-    (drawings 22)
+    (drawings 24)
     (tracks 63)
     (zones 0)
@@
   )
   (module MRDT_Silkscreens:MRDT_Logo_7.5mm (layer F.Cu)
-    (at 150.114 96.774)
+    (at 149.86 95.504)
     (tags "Logo, MRDT")
     (fp_text reference G*** (at -1.0922 4.2418) (layer Dwgs.User) hide
@@
       (xy 2.655043 -6.074854) (xy 2.83052 -6.086745) (xy 3.000245 -6.084745)) (layer F.SilkS) (width 0.01))
   )
+  (gr_text Off (at 153.67 100.838) (layer F.SilkS)
+    (effects (font (size 1.5 1.5) (thickness 0.3)))
+  )
+  (gr_text On (at 153.67 91.44) (layer F.SilkS)
+    (effects (font (size 1.5 1.5) (thickness 0.3)))
+  )
   (gr_text "Wireless E-Stop Reciever Rev.1\nMars Rover, Valkyrie\nMissouri S&T \nAndrew Simily" (at 134.112 97.028) (layer B.SilkS)

Commit message: Adjusted things & made Gerbs
Parts:
- moved G*** 4.95 mm to (127.4, 102.7)
- moved R1 4.95 mm to (142.2, 99.2), turned to 0 degrees
- moved D1 4.84 mm to (137.3, 99.1), turned to 180 degrees
- moved G*** 1.02 mm to (149.4, 96.4)
- turned D3 to 180 degrees
- renumbered PWR_SW1 to POWER
Routing:
- net Net-(D3-Pad1): track 6.71 -> 3.09 mm
- net +3V3: track 49.7 -> 48.0 mm
- net Net-(D1-Pad2): track 35.1 -> 34.1 mm
Other:
- outline, holes or cut-outs redrawn
