File: WirelessEStop_Tx.sch (KiCad schematic (older format))
At the start: 10 parts

Commit message: This bout to be some dope shiz
Parts:
- removed Conn?: 9V Batt, symbol MRDT_Connectors:Molex_SL_02
- removed D?: LED, symbol Device:LED
- removed R? (x3): 10K, symbol Device:R
- removed SW?: Master Power, symbol Switch:SW_SPST
- removed SW?: Maintain Switch, symbol Switch:SW_SPST
- removed SW?: MOM Switch, symbol Switch:SW_Push
- removed U?: OKI_3V3, symbol MRDT_Devices:OKI
- removed U?: ESP_8266_01, symbol ESP_8266_01:ESP_8266_01
- added C?: C, symbol Device:C
- added C?: 2.4pF, symbol Device:C
- added C?: 3.0pF, symbol Device:C
- added J?: U.FL-R-SMT(01), HRS_U.FL-R-SMT(01), symbol U.FL-R-SMT_01_:U.FL-R-SMT(01)
- added J?: USB_C_Receptacle, symbol Connector:USB_C_Receptacle
- added J? (x3): Conn_01x02, symbol Connector_Generic:Conn_01x02
- added L?: 2.2nH, symbol pspice:INDUCTOR
- added R?: 12k, symbol Device:R
- added R? (x6): 200, symbol Device:R
- added SW?: SW_Push, symbol Switch:SW_Push
- added SW?: SW_DIP_x02, symbol Switch:SW_DIP_x02
- added U?: ESP8266EX, symbol ESP8266:ESP8266EX
- added U?: CH340, MSOP10-NOPAD, symbol CH340:CH340
- added U?: MCP73833-BZI_UN, SOP50P490X110-10N, symbol MCP73833-BZI_UN:MCP73833-BZI_UN
Connections:
- net labels added: +3.3V, +BATT, Charger_IND_1, Charger_IND_2, Charger_IND_PG, D+, D-, RXD, Reset, SD_CLK, SD_CMD, SD_D0, SD_D1, SD_D2, SD_D3, TXD
- net labels removed: +3V3, Vin
- wire segments 16 -> 66
- no-connect marks 0 -> 18
Other:
- note added: "Battery Charger & Regulator"
- note added: "Battery Connector"
- note added: "Esp Connections"
- note added: "Externally Connected Components"
- note added: "Indicators"
- note added: "On/Off Switch"
- note added: "Thermistor for battery"
- note added: "UART Rx, Tx Converter"
- note added: "USB-C Port"

Commit message: What the fuck did you just fucking say about me, you little bitch? I'll have you know I graduated top of my class in the Navy Seals, and I've been involved in numerous secret raids on Al-Quaeda, and I have over 300 confirmed kills. I am trained in gorilla warfare and I'm the top sniper in the entire US armed forces. You are nothing to me but just another target. I will wipe you the fuck out with precision the likes of which has never been seen before on this Earth, mark my fucking words. You think you can get away with saying that shit to me over the Internet? Think again, fucker. As we speak I am contacting my secret network of spies across the USA and your IP is being traced right now so you better prepare for the storm, maggot. The storm that wipes out the pathetic little thing you call your life. You're fucking dead, kid. I can be anywhere, anytime, and I can kill you in over seven hundred ways, and that's just with my bare hands. Not only am I extensively trained in unarmed combat, but I have access to the entire arsenal of the United States Marine Corps and I will use it to its full extent to wipe your miserable ass off the face of the continent, you little shit. If only you could have known what unholy retribution your little "clever" comment was about to bring down upon you, maybe you would have held your fucking tongue. But you couldn't, you didn't, and now you're paying the price, you goddamn idiot. I will shit fury all over you and you will drown in it. You're fucking dead, kiddo
Parts:
- removed SW?: SW_DIP_x02, symbol Switch:SW_DIP_x02
- added J?: Conn_01x02, symbol Connector_Generic:Conn_01x02
Other:
- moved on the sheet: SW?
Changed lines of the file:
@@
 Wire Wire Line
 	10200 5050 10250 5050
-Text GLabel 10250 4950 2    39   Output ~ 0
+Text GLabel 10250 4950 2    39   Input ~ 0
 Charger_IND_1
-Text GLabel 10250 5050 2    39   Output ~ 0
+Text GLabel 10250 5050 2    39   Input ~ 0
 Charger_IND_2
 Text GLabel 8550 5050 0    39   Output ~ 0
@@
 L Switch:SW_Push SW?
 U 1 1 5DEE0F97
-P 2550 5300
-F 0 "SW?" H 2550 5585 50  0000 C CNN
-F 1 "SW_Push" H 2550 5494 50  0000 C CNN
-F 2 "" H 2550 5500 50  0001 C CNN
-F 3 "~" H 2550 5500 50  0001 C CNN
-	1    2550 5300
-	1    0    0    -1
-$EndComp
-$Comp
-L Switch:SW_DIP_x02 SW?
-U 1 1 5DEE2995
-P 3800 5300
-F 0 "SW?" H 3800 5667 50  0000 C CNN
-F 1 "SW_DIP_x02" H 3800 5576 50  0000 C CNN
-F 2 "" H 3800 5300 50  0001 C CNN
-F 3 "~" H 3800 5300 50  0001 C CNN
-	1    3800 5300
+P 2300 5050
+F 0 "SW?" H 2300 5335 50  0000 C CNN
+F 1 "SW_Push" H 2300 5244 50  0000 C CNN
+F 2 "" H 2300 5250 50  0001 C CNN
+F 3 "~" H 2300 5250 50  0001 C CNN
+	1    2300 5050
 	1    0    0    -1
 $EndComp
@@
 	1250 5050 1550 5050
 NoConn ~ 6050 3050
+$Comp
+L Connector_Generic:Conn_01x02 J?
+U 1 1 5DF7A0B6
+P 800 5600
+F 0 "J?" V 800 5350 50  0000 C CNN
+F 1 "Conn_01x02" V 950 5250 50  0000 L CNN
+F 2 "" H 800 5600 50  0001 C CNN
+F 3 "~" H 800 5600 50  0001 C CNN
+	1    800  5600
+	0    -1   -1   0
+$EndComp
 $EndSCHEMATC

Commit message: Bee Movie Script - Dialogue Transcript     According to all known laws of aviation,     there is no way a bee should be able to fly.     Its wings are too small to get its fat little body off the ground.     The bee, of course, flies anyway     because bees don't care what humans think is impossible.     Yellow, black. Yellow, black. Yellow, black. Yellow, black.     Ooh, black and yellow! Let's shake it up a little.     Barry! Breakfast is ready!     Ooming!     Hang on a second.     Hello?     - Barry? - Adam?     - Oan you believe this is happening? - I can't. I'll pick you up.     Looking sharp.     Use the stairs. Your father paid good money for those.     Sorry. I'm excited.     Here's the graduate. We're very proud of you, son.     A perfect report card, all B's.     Very proud.     Ma! I got a thing going here.     - You got lint on your fuzz. - Ow! That's me!     - Wave to us! We'll be in row 118,000. - Bye!     Barry, I told you, stop flying in the house!     - Hey, Adam. - Hey, Barry.     - Is that fuzz gel? - A little. Special day, graduation.     Never thought I'd make it.     Three days grade school, three days high school.     Those were awkward.     Three days college. I'm glad I took a day and hitchhiked around the hive.     You did come back different.     - Hi, Barry. - Artie, growing a mustache? Looks good.     - Hear about Frankie? - Yeah.     - You going to the funeral? - No, I'm not going.     Everybody knows, sting someone, you die.     Don't waste it on a squirrel. Such a hothead.     I guess he could have just gotten out of the way.     I love this incorporating an amusement park into our day.     That's why we don't need vacations.     Boy, quite a bit of pomp... under the circumstances.     - Well, Adam, today we are men. - We are!     - Bee-men. - Amen!     Hallelujah!     Students, faculty, distinguished bees,     please welcome Dean Buzzwell.     Welcome, New Hive Oity graduating class of...     ...9:15.     That concludes our ceremoni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
Parts:
- added C? (x2): 10pF, symbol Device:C
- added C? (x2): .1uF, symbol Device:C
- added R?: 10k, symbol Device:R
- added U?: 25Q128FV, symbol 25Q128FV:25Q128FV
- added Y?: Crystal_GND24, symbol Device:Crystal_GND24
Connections:
- net +3V3: now also C?.1, C?.1, R?.2, U?.8 (Vcc)
- net GND: now also C?.1, C?.1, C?.2, U?.4 (GND), Y?.2, Y?.4
- net SD_CLK: now also U?.6 (CLK)
- net SD_CMD: now also U?.1 (/CS)
- net SD_D0: now also U?.5 (DI(I/O_0))
- net SD_D1: now also U?.2 (DO(I/O_1))
- net SD_D2: now also U?.7 (I/O_3)
- net SD_D3: now also U?.3 (/WP(I/O_2))
- net at U?.1 (VddA), U?.3 (Vdd3P3), U?.4 (Vdd3P3): now also C?.1, L?.2, U?.2 (LNA/ANT); no longer U?.7 (CHIP_EN), U?.8 (XPD_DCDC)
- net at U?.27 (XTAL_OUT): now also C?.2, Y?.3
- net at U?.28 (XTAL_IN): now also C?.2, Y?.1
- net at U?.7 (7-VCC): now also C?.2
- new net: R?.1, U?.7 (CHIP_EN)
Other:
- note added: "Flash Memory"
- note added: "Toggle Power"
- moved on the sheet: C?, J?, L?, R?, SW?, U?

Commit message: if(reader == "Eli") print("Get Fucked")
Parts:
- removed C?: .1uF, symbol Device:C
- removed J?: USB_C_Receptacle, symbol Connector:USB_C_Receptacle
- removed J? (x3): Conn_01x02, symbol Connector_Generic:Conn_01x02
- removed U?: MCP73833-BZI_UN, SOP50P490X110-10N, symbol MCP73833-BZI_UN:MCP73833-BZI_UN
- added C7: 10nF, symbol Device:C
- added C8: 10uF, symbol Device:C
- added D1, D2, D3, D4: D, symbol Device:D
- added J3: USB_B_Micro, symbol Connector:USB_B_Micro
- added Q1: Q_NMOS_GSD, symbol Device:Q_NMOS_GSD
- added R12, R15: 330, symbol Device:R
- added R13: 500, symbol Device:R
- added R14, R2, R3: 1k, symbol Device:R
- added R16, R17: 470, symbol Device:R
- added R18: 2k, symbol Device:R
- added R4: 10k, symbol Device:R
- added SW2, SW5: SW_DIP_x01, symbol Switch:SW_DIP_x01
- added SW4, SW?: SW_Push, symbol Switch:SW_Push
- added SW?: SW_SPDT, symbol Switch:SW_SPDT
- added U4: MCP73831T-2ACI_OT, SOT95P280X145-5N, symbol MCP73831T-2ACI_OT:MCP73831T-2ACI_OT
- gave numbers to parts that had none: 22
Connections:
- net +3V3: now also SW3.1, SW3.2, U3.10 (10-V3), U3.7 (7-VCC), R2.2, R3.2, R4.2, SW?.1, SW?.1 (A)
- net +BATT: now also J2.2 (Pin_2), SW2.1, U4.3 (VBAT)
- net D+: now also J3.3 (D+)
- net D-: now also J3.2 (D-)
- net GND: now also C7.1, C8.2, D1.1 (K), D2.1 (K), J3.5 (GND), Q1.2 (S), R15.2, R17.2, R18.1, R4.1, SW5.2, SW?.2, U4.2 (VSS)
- net at U1.1 (VddA), U1.3 (Vdd3P3), U1.4 (Vdd3P3): no longer C3.1, L1.2, U1.2 (LNA/ANT)
- net IND_LowBattery: now reaches U1.10 (MTDI/GPIO12)
- net IND_LowBattery: now also R12.2
- net IND_Connected: now reaches U1.12 (MTCK/GPIO13)
- net IND_Arm: now reaches U1.13 (MTDO/GPIO15)
- net I2C_SDA: now reaches U1.14 (GPIO2)
- net SW_Flash: now reaches U1.15 (GPIO0)
- net SW_Flash: now also SW5.1
- net SW_Trigger: now reaches U1.16 (GP4/VD)
- net SW_Trigger: now also SW?.2 (B)
- net SW_Arm: now reaches U1.24 (GP5/VD)
- net ADC_In: now reaches U1.6 (TOUT)
- net ADC_In: now also C7.2, R14.1, R15.1
- net I2C_CLK: now reaches U1.9 (MTMS/GPIO14)
- new net: C3.1, L1.2, U1.2 (LNA/ANT)
- new net: D3.2 (A), R16.2
- new net: D4.1 (K), R17.1
- new net: Q1.3 (D), R2.1, SW?.3 (C)
- new net: Q1.1 (G), R3.1
- new net: D1.2 (A), R12.1
- new net: D2.2 (A), R13.1
- new net ADC_VDiv: R14.2, SW2.2
- new net DC_In: C8.1, J3.1 (VBUS), R13.2, R16.1, U4.4 (VDD)
- new net Prog_Out: R18.2, U4.5 (PROG)
- new net Stat_Out: D3.1 (K), D4.2 (A), U4.1 (STAT)
- no-connect marks 18 -> 5
Other:
- note added: "5V Supply"
- note added: "Arm/Connect Button"
- note added: "Batt Regulator"
- note added: "Batt V ADC"
- note added: "Battery Charger"
- note added: "Charger Control Resistor"
- note added: "Flash Mode"
- note added: "Green LED"
- note added: "Green LED\nCharged"
- note added: "Haptic Feedback"
- note added: "I/O Components"
- note added: "Micro-USB Port"
- note added: "Red LED\nCharging"
- note added: "Reset Button"
- note added: "Toggle Active High/Low"
- note added: "Trigger Button"
- note removed: "Battery Charger & Regulator"
- note removed: "Externally Connected Components"
- note removed: "On/Off Switch"
- note removed: "Thermistor for battery"
- note removed: "USB-C Port"
- moved on the sheet: C1, C2, C3, C4, C5, C6, J1, J2, L1, R1, R10, R11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

Commit message: Schematic is done, nothing snarky to say other than I'm the fuckin best
Parts:
- removed R10, R11, R6, R7, R9: 200, symbol Device:R
- added C? (x2): 1uF, symbol Device:C
- added C? (x2): .1uF, symbol Device:C
- added C?: 10uF, symbol Device:C
- added D? (x13): D, symbol Device:D
- added IC?: DRV2605LDGSR, SOP50P490X110-10N, symbol DRV2605LDGSR:DRV2605LDGSR
- added J?: Conn_01x02, symbol Connector_Generic:Conn_01x02
- added R?: 30.1k, symbol Device:R
- added R?: 52.3k, symbol Device:R
- added R? (x2): 2.2k, symbol Device:R
- added R?: 10k, symbol Device:R
- added R? (x13): 330, symbol Device:R
- added U?: TPS73633DBVR, SOT95P280X145-5N, symbol TPS73633DBVR:TPS73633DBVR
Connections:
- net Reset is gone; now on net SW_Reset: U1.32 (EXT_RSTB)
- net +3V3: now also C?.1, C?.1, C?.1, C?.1, IC?.10 (VDD), IC?.5 (EN), R?.1, R?.2, R?.2, R?.2, R?.2, U?.5 (OUT); no longer R3.2, R4.2, SW3.1, SW?.1 (A)
- net ADC_VDiv: now also U?.1 (IN), U?.3 (EN)
- net GND: now also SW4.2, C?.2, C?.2, C?.2, D?.1 (K), D?.1 (K), D?.1 (K), D?.1 (K), D?.1 (K), D?.1 (K), D?.1 (K), D?.1 (K), D?.1 (K), D?.1 (K), D?.1 (K), D?.1 (K), D?.1 (K), IC?.8 (GND), R?.2, U?.2 (GND)
- net I2C_CLK: now also IC?.2 (SCL), R?.1, R?.2
- net I2C_SDA: now also IC?.3 (SDA), R?.1, R?.2
- net IND_Arm: now also R?.2
- net IND_Connected: now also R?.2
- net RXD: now also R?.2
- net SD_CMD: now also U1.20 (SD_CMD), R?.2; no longer U2.1 (/CS)
- net SD_D0: now also U1.22 (SD_D0)
- net SD_D1: now also U1.23 (SD_D1)
- net SD_D2: now also U1.18 (SD_D2)
- net SD_D3: now also U1.19 (SD_D3)
- net SW_Flash: now also R?.2
- net SW_Trigger: now also R?.2
- net TXD: now also R?.2
- net at U1.1 (VddA), U1.3 (Vdd3P3), U1.4 (Vdd3P3): now also C?.2, C?.2
- net IND_Software: now reaches U1.8 (XPD_DCDC)
- net IND_Software: now also R?.2
- net SW_Reset: now reaches SW4.1
- net SW_Reset: now also R?.1, R?.2
- new net: R3.2, R4.2, SW3.1, SW?.1 (A)
- new net: R?.1, R?.2, U?.4 (NR/FB)
- new net: C?.1, IC?.1 (REG)
- new net: D?.2 (A), R?.1 (x13)
- new net Motor+: IC?.7 (OUT+), J?.1 (Pin_1), R?.2
- new net Motor-: IC?.9 (OUT-), J?.2 (Pin_2)
- no-connect marks 5 -> 8
Other:
- note added: "Battery"
- note added: "Blue LED"
- note added: "Haptic Motor"
- note added: "Orange LED"
- note added: "Pink LED"
- note added: "Red LED"
- note added: "Yellow LED"
- note removed: "Battery Connector"
- moved on the sheet: C1, C2, C3, C4, C5, C6, C7, D1, D2, J1, J2, J3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

Commit message: commit kiddos
Parts:
- C1, C2, C3, C4, C5, C6, C7, C8: footprint (none) -> Capacitor_SMD:C_0603_1608Metric_Pad1.05x0.95mm_HandSolder
- C10, C11, C12, C13, C9: renamed from C?; footprint (none) -> Capacitor_SMD:C_0603_1608Metric_Pad1.05x0.95mm_HandSolder
- D1, D2, D3, D4: footprint (none) -> LED_SMD:LED_0603_1608Metric_Pad1.05x0.95mm_HandSolder
- D10, D11, D12, D13, D14, D15, D16, D17, D5, D6, D7, D8, D9: renamed from D?; footprint (none) -> LED_SMD:LED_0603_1608Metric_Pad1.05x0.95mm_HandSolder
- IC1: renamed from IC?; footprint SOP50P490X110-10N -> DRV2605LDGSR:SOP50P490X110-10N
- J1: footprint HRS_U.FL-R-SMT(01) -> U.FL-R-SMT_01_:HRS_U.FL-R-SMT(01)
- J2: footprint (none) -> Connector_JST:JST_EH_S2B-EH_1x02_P2.50mm_Horizontal
- J3: footprint (none) -> Connector_USB:USB_Micro-B_Amphenol_10103594-0001LF_Horizontal
- J4: renamed from J?; footprint (none) -> Connector_JST:JST_EH_S2B-EH_1x02_P2.50mm_Horizontal
- L1: footprint (none) -> Inductor_SMD:L_0603_1608Metric_Pad1.05x0.95mm_HandSolder
- R1, R12, R13, R14, R15, R16, R17, R18, R2, R3, R4, R5, R8: footprint (none) -> Resistor_SMD:R_0603_1608Metric_Pad1.05x0.95mm_HandSolder
- R10, R11, R19, R20, R21, R22, R23, R24, R25, R26, R27, R28, R29, R30, R31, R6, R7, R9: renamed from R?; footprint (none) -> Resistor_SMD:R_0603_1608Metric_Pad1.05x0.95mm_HandSolder
- SW1: renamed from SW?; footprint (none) -> Button_Switch_SMD:SW_Push_1P1T_NO_CK_PTS125Sx43PSMTR
- SW3, SW4: footprint (none) -> Button_Switch_SMD:SW_Push_1P1T_NO_CK_PTS125Sx43PSMTR
- U1: footprint (none) -> ESP8266:ESP2866EX_Chip
- U2: footprint (none) -> W25Q128FVSIF:SOIC127P600X175-8N
- U3: footprint MSOP10-NOPAD -> CH340E:MSOP10
- Y1: footprint (none) -> Crystal:Crystal_SMD_2016-4Pin_2.0x1.6mm
- gave numbers to parts that had none: 2
Connections:
- net SD_CMD: now also U2.1 (/CS)
Other:
- moved on the sheet: C1, C10, C11, C2, C3, C4, C5, C6, C9, J1, L1, R1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

Commit message: If you can read this message, please, you need to do something. I'm locked in the github server room, and the things I've seen.... Oh fuck, I think I hear a comp sci coming OH GOD PLEASE NO, HEL......
Parts:
- removed C4: C, Capacitor_SMD:C_0603_1608Metric_Pad1.05x0.95mm_HandSolder, symbol Device:C
- removed D12, D13: D, LED_SMD:LED_0603_1608Metric_Pad1.05x0.95mm_HandSolder, symbol Device:D
- removed R24, R25: 330, Resistor_SMD:R_0603_1608Metric_Pad1.05x0.95mm_HandSolder, symbol Device:R
- removed SW1: SW_Push, Button_Switch_SMD:SW_Push_1P1T_NO_CK_PTS125Sx43PSMTR, symbol Switch:SW_Push
- added SW1: SW_DIP_x01, Button_Switch_THT:SW_CuK_JS202011CQN_DPDT_Straight, symbol Switch:SW_DIP_x01
- SW2, SW5: footprint (none) -> Button_Switch_THT:SW_CuK_JS202011CQN_DPDT_Straight
- SW3, SW4: footprint Button_Switch_SMD:SW_Push_1P1T_NO_CK_PTS125Sx43PSMTR -> Button_Switch_SMD:SW_SPST_TL3305A
Connections:
- net +3V3: now also R21.2, R23.2, R26.2, U1.29 (VDDD), U1.30 (VDDA)
- net GND: no longer D11.1 (K), D14.1 (K), D9.1 (K)
- net I2C_SDA: now also D14.1 (K); no longer R26.2
- net SD_CMD: now also D9.1 (K)
- net SW_Flash: now also D11.1 (K); no longer R23.2
- net SW_Reset: no longer R21.2
Other:
- note added: "Arm Switch"
- note removed: "Arm/Connect Button"
- moved on the sheet: D1, D11, D14, D16, D17, D2, D6, D7, D8, D9, R11, R12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

Commit message: Eli suck my dick
Connections:
- net +3V3: no longer U1.29 (VDDD), U1.30 (VDDA)
- net at C10.2, C11.2, U1.1 (VddA)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: now also U1.29 (VDDD), U1.30 (VDDA)
Changed lines of the file:
@@
-$EndComp
-$Comp
-L power:+3.3V #PWR013
-U 1 1 5DE96AF6
-P 3550 1850
-F 0 "#PWR013" H 3550 1700 50  0001 C CNN
-F 1 "+3.3V" H 3565 2023 50  0000 C CNN
-F 2 "" H 3550 1850 50  0001 C CNN
-F 3 "" H 3550 1850 50  0001 C CNN
-	1    3550 1850
-	1    0    0    -1
 $EndComp
 $Comp
@@
 Text Notes 7750 5900 1    30   ~ 0
 Pink LED
+Wire Wire Line
+	3550 1850 2400 1850
+Wire Wire Line
+	2400 1850 2400 2400
 $EndSCHEMATC
