File: WirelessEStop_Tx.sch (KiCad schematic (older format))
At the start: 75 parts, among them IC1 DRV2605LDGSR, J1 U.FL-R-SMT(01), J2 Conn_01x02, J3 USB_B_Micro, J4 Conn_01x02, Q1 Q_NMOS_GSD, SW1 SW_DIP_x01, SW2 SW_DIP_x01, SW3 SW_Push, SW4 SW_Push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

Commit message: Please let the sweet release of death take me soon
Parts:
- Q1: footprint (none) -> IRLML6344TRPBF:SOT95P240X112-3N
- SW1: footprint Button_Switch_THT:SW_CuK_JS202011CQN_DPDT_Straight -> Button_Switch_THT:SW_CuK_JS202011AQN_DPDT_Angled
- SW6: footprint (none) -> MRDT_Switches:1P2T_Angled_Slide_GPI-152-3013
- U4, U5: footprint SOT95P280X145-5N -> (none)
Connections:
- net +3V3: now also SW1.1
- net IND_Arm: no longer R19.2
- net IND_Connected: now also U1.8 (XPD_DCDC); no longer U1.12 (MTCK/GPIO13)
- net IND_Software: now also U1.12 (MTCK/GPIO13); no longer U1.8 (XPD_DCDC)
- net SW_Arm: now also R19.2, SW1.2
Other:
- moved on the sheet: C10, C11, SW1

Commit message: l
Parts:
- R18: value 2k -> 2k2
Connections:
- net +3V3: now also U1.1 (VddA), U1.29 (VDDD), U1.3 (Vdd3P3), U1.30 (VDDA), U1.4 (Vdd3P3)
- net GND: now also C10.2, C11.2
- net RXD: now also R27.2, U1.26 (UTXD); no longer R28.2, U1.25 (URXD)
- net TXD: now also R28.2, U1.25 (URXD); no longer R27.2, U1.26 (UTXD)
Other:
- note added: "Arming Switch"
- note added: "Dan Napierkowski"
- note added: "Software Flash"
- note removed: "Arm Switch"
- note removed: "Flash Mode"
- moved on the sheet: C10, C11
Changed lines of the file:
@@
 Wire Wire Line
 	9900 1600 9950 1600
-Text GLabel 9950 1500 2    39   Output ~ 0
+Text GLabel 9950 1500 2    39   Input ~ 0
 RXD
 Text GLabel 9950 1600 2    39   Output ~ 0
@@
 	1    0    0    -1
 $EndComp
-Text GLabel 3900 1900 1    39   Input ~ 0
-TXD
-Text GLabel 4000 1900 1    39   Input ~ 0
-RXD
 Wire Wire Line
 	3900 1950 3900 1900
@@
 P 10350 4050
 F 0 "R18" V 10250 4050 50  0000 C CNN
-F 1 "2k" V 10350 4050 50  0000 C CNN
+F 1 "2k2" V 10350 4050 50  0000 C CNN
 F 2 "Resistor_SMD:R_0603_1608Metric_Pad1.05x0.95mm_HandSolder" V 10280 4050 50  0001 C CNN
 F 3 "~" H 10350 4050 50  0001 C CNN
@@
 U 1 1 5E381E5E
 P 2350 5600
-F 0 "R3" V 2250 5600 50  0000 C CNN
+F 0 "R3" H 2250 5600 50  0000 C CNN
 F 1 "1k" V 2350 5600 50  0000 C CNN
 F 2 "Resistor_SMD:R_0603_1608Metric_Pad1.05x0.95mm_HandSolder" V 2280 5600 50  0001 C CNN
@@
 U 1 1 5E388BBF
 P 2550 5600
-F 0 "R4" V 2450 5600 50  0000 C CNN
+F 0 "R4" H 2450 5600 50  0000 C CNN
 F 1 "10k" V 2550 5600 50  0000 C CNN
 F 2 "Resistor_SMD:R_0603_1608Metric_Pad1.05x0.95mm_HandSolder" V 2480 5600 50  0001 C CNN
@@
 Wire Wire Line
 	2350 5400 2450 5400
-Wire Wire Line
-	2450 5150 2450 5400
 Connection ~ 2450 5400
 Wire Wire Line
@@
 $EndComp
 Wire Wire Line
-	1700 5250 1900 5250
-Wire Wire Line
-	1900 5250 1900 5150
-Wire Wire Line
 	1700 5450 1900 5450
 Wire Wire Line
@@
 U 1 1 5E342249
 P 2000 5350
-F 0 "R2" V 1900 5350 50  0000 C CNN
+F 0 "R2" H 1900 5350 50  0000 C CNN
 F 1 "1k" V 2000 5350 50  0000 C CNN
 F 2 "Resistor_SMD:R_0603_1608Metric_Pad1.05x0.95mm_HandSolder" V 1930 5350 50  0001 C CNN
@@
 Wire Wire Line
 	2900 1250 3300 1250
-$Comp
-L power:+3.3V #PWR037
-U 1 1 5F784180
-P 1900 1950
-F 0 "#PWR037" H 1900 1800 50  0001 C CNN
-F 1 "+3.3V" H 2000 2100 50  0000 R CNN
-F 2 "" H 1900 1950 50  0001 C CNN
-F 3 "" H 1900 1950 50  0001 C CNN
-	1    1900 1950
-	1    0    0    -1
-$EndComp
-$Comp
-L Device:C C10
-U 1 1 5F784817
-P 1900 2200
-F 0 "C10" H 1700 2200 50  0000 L CNN
-F 1 "10uF" H 1650 2100 50  0000 L CNN
-F 2 "Capacitor_SMD:C_0603_1608Metric_Pad1.05x0.95mm_HandSolder" H 1938 2050 50  0001 C CNN
-F 3 "~" H 1900 2200 50  0001 C CNN
-	1    1900 2200
-	1    0    0    -1
-$EndComp
-$Comp
-L Device:C C11
-U 1 1 5F784F3D
-P 2250 2200
-F 0 "C11" H 2050 2200 50  0000 L CNN
-F 1 ".1uF" H 2000 2100 50  0000 L CNN
-F 2 "Capacitor_SMD:C_0603_1608Metric_Pad1.05x0.95mm_HandSolder" H 2288 2050 50  0001 C CNN
-F 3 "~" H 2250 2200 50  0001 C CNN
-	1    2250 2200
-	1    0    0    -1
-$EndComp
-Wire Wire Line
-	1900 1950 1900 2000
-Wire Wire Line
-	1900 2000 2250 2000
-Wire Wire Line
-	2250 2000 2250 2050
-Connection ~ 1900 2000
-Wire Wire Line
-	1900 2000 1900 2050
 Connection ~ 2400 2400
 Wire Wire Line
@@
 SW_Flash
 Text Notes 2300 7100 0    79   ~ 16
-Flash Mode
+Software Flash
 $Comp
 L Switch:SW_DIP_x01 SW5
@@
 Wire Notes Line
 	3500 4300 3500 7900
-Wire Wire Line
-	1900 5150 2450 5150
 Text GLabel 3150 6750 2    39   Output ~ 0
 Reg_In
@@
 Toggle Power
 Text Notes 550  6400 0    79   ~ 16
-Arm Switch
+Arming Switch
 Wire Notes Line
 	6967 6537 5701 6537
@@
 Wire Wire Line
 	8200 5800 8200 5700
-Wire Wire Line
-	8200 5400 8200 5300
 $Comp
 L Device:R R27
@@
 	8450 5800 8450 5700
 Wire Wire Line
-	8450 5400 8450 5300
+	8200 5400 8200 5300
 $Comp
 L Device:R R28
@@
 Motor+
 Text GLabel 8200 5300 1    39   Input ~ 0
-TXD
-Text GLabel 8450 5300 1    39   Input ~ 0
 RXD
 Text GLabel 6450 5300 1    39   Input ~ 0
@@
 Connection ~ 3500 1900
 Wire Wire Line
-	3500 1900 3550 1900
-Wire Wire Line
 	3500 1900 3600 1900
-Wire Wire Line
-	1900 2350 1900 2400
-Wire Wire Line
-	1900 2400 2250 2400
-Wire Wire Line
-	2250 2350 2250 2400
-Connection ~ 2250 2400
-Wire Wire Line
-	2250 2400 2400 2400
 Text GLabel 6700 5300 1    39   Input ~ 0
 SW_Arm
+Wire Wire Line
+	1850 5250 1850 4950
+Wire Wire Line
+	1850 4950 2450 4950
+Wire Wire Line
+	2450 4950 2450 5400
+Wire Wire Line
+	1700 5250 1850 5250
+Text Notes 7750 7000 0    197  ~ 39
+Dan Napierkowski
+Wire Wire Line
+	1550 1900 1550 1950
+$Comp
+L Device:C C11
+U 1 1 5F784F3D
+P 1850 2100
+F 0 "C11" H 1850 2200 50  0000 L CNN
+F 1 ".1uF" H 1850 2000 50  0000 L CNN
+F 2 "Capacitor_SMD:C_0603_1608Metric_Pad1.05x0.95mm_HandSolder" H 1888 1950 50  0001 C CNN
+F 3 "~" H 1850 2100 50  0001 C CNN
+	1    1850 2100
+	1    0    0    -1
+$EndComp
+$Comp
+L Device:C C10
+U 1 1 5F784817
+P 1550 2100
+F 0 "C10" H 1550 2200 50  0000 L CNN
+F 1 "10uF" H 1550 2000 50  0000 L CNN
+F 2 "Capacitor_SMD:C_0603_1608Metric_Pad1.05x0.95mm_HandSolder" H 1588 1950 50  0001 C CNN
+F 3 "~" H 1550 2100 50  0001 C CNN
+	1    1550 2100
+	1    0    0    -1
+$EndComp
+$Comp
+L power:+3.3V #PWR037
+U 1 1 5F784180
+P 1850 1850
+F 0 "#PWR037" H 1850 1700 50  0001 C CNN
+F 1 "+3.3V" H 1950 2000 50  0000 R CNN
+F 2 "" H 1850 1850 50  0001 C CNN
+F 3 "" H 1850 1850 50  0001 C CNN
+	1    1850 1850
+	1    0    0    -1
+$EndComp
+Text GLabel 4000 1900 1    39   Input ~ 0
+TXD
+Text GLabel 3900 1900 1    39   Output ~ 0
+RXD
+Connection ~ 2400 1900
+Wire Wire Line
+	1850 1950 1850 1900
+Connection ~ 1850 1900
+Wire Wire Line
+	1850 1900 1550 1900
+Wire Wire Line
+	1550 2250 1550 2300
+Wire Wire Line
+	1850 2300 1850 2250
+$Comp
+L power:GND #PWR0105
+U 1 1 5E41225D
+P 2200 2350
+F 0 "#PWR0105" H 2200 2100 50  0001 C CNN
+F 1 "GND" H 2100 2250 50  0000 C CNN
+F 2 "" H 2200 2350 50  0001 C CNN
+F 3 "" H 2200 2350 50  0001 C CNN
+	1    2200 2350
+	1    0    0    -1
+$EndComp
+Wire Wire Line
+	1550 2300 1850 2300
+Wire Wire Line
+	1850 2300 2200 2300
+Wire Wire Line
+	2200 2300 2200 2350
+Connection ~ 1850 2300
+Wire Wire Line
+	1850 1900 2400 1900
+Wire Wire Line
+	1850 1900 1850 1850
+Text GLabel 8450 5300 1    39   Input ~ 0
+TXD
+Wire Wire Line
+	8450 5400 8450 5300
 $EndSCHEMATC

Commit message: Rethinkimg things
Parts:
- IC1: symbol DRV2605LDGSR:DRV2605LDGSR -> WirelessEStop_Tx-rescue:DRV2605LDGSR-DRV2605LDGSR
- J1: symbol U.FL-R-SMT_01_:U.FL-R-SMT(01) -> WirelessEStop_Tx-rescue:U.FL-R-SMT(01)-U.FL-R-SMT_01_
- U1: symbol ESP8266:ESP8266EX -> WirelessEStop_Tx-rescue:ESP8266EX-ESP8266
- U2: symbol 25Q128FV:25Q128FV -> WirelessEStop_Tx-rescue:25Q128FV-25Q128FV
- U3: symbol CH340:CH340 -> WirelessEStop_Tx-rescue:CH340-CH340
- U4: symbol MCP73831T-2ACI_OT:MCP73831T-2ACI_OT -> WirelessEStop_Tx-rescue:MCP73831T-2ACI_OT-MCP73831T-2ACI_OT
- U5: symbol TPS73633DBVR:TPS73633DBVR -> WirelessEStop_Tx-rescue:TPS73633DBVR-TPS73633DBVR
Connections:
- net IND_Arm: no longer names the net of U1.13 (MTDO/GPIO15)
- no-connect marks 8 -> 9
Changed lines of the file:
@@
 EESchema Schematic File Version 4
+LIBS:WirelessEStop_Tx-cache
 EELAYER 30 0
 EELAYER END
@@
 $EndDescr
 $Comp
-L U.FL-R-SMT_01_:U.FL-R-SMT(01) J1
+L WirelessEStop_Tx-rescue:U.FL-R-SMT(01)-U.FL-R-SMT_01_ J1
 U 1 1 5DE8D7E8
 P 1100 2100
@@
 Micro-USB Port
 $Comp
-L CH340:CH340 U3
+L WirelessEStop_Tx-rescue:CH340-CH340 U3
 U 1 1 5DEA79E8
 P 9300 1600
@@
 Indicators
 $Comp
-L 25Q128FV:25Q128FV U2
+L WirelessEStop_Tx-rescue:25Q128FV-25Q128FV U2
 U 1 1 5DEF0BBC
 P 6650 3450
@@
 	400  850  11300 850
 $Comp
-L MCP73831T-2ACI_OT:MCP73831T-2ACI_OT U4
+L WirelessEStop_Tx-rescue:MCP73831T-2ACI_OT-MCP73831T-2ACI_OT U4
 U 1 1 5DFCDF8F
 P 9650 3200
@@
 	3800 3800 4050 3800
 Wire Wire Line
-	3700 3550 3700 3900
-Wire Wire Line
-	3700 3900 4050 3900
-Text GLabel 4050 3900 2    39   Output ~ 0
-IND_Arm
-Wire Wire Line
 	3500 3550 3500 3850
 Wire Wire Line
@@
 SW_Arm
 $Comp
-L TPS73633DBVR:TPS73633DBVR U5
+L WirelessEStop_Tx-rescue:TPS73633DBVR-TPS73633DBVR U5
 U 1 1 5EB322E2
 P 10150 5450
@@
 $EndComp
 $Comp
-L DRV2605LDGSR:DRV2605LDGSR IC1
+L WirelessEStop_Tx-rescue:DRV2605LDGSR-DRV2605LDGSR IC1
 U 1 1 5ECF13D4
 P 3800 5800
@@
 IND_Software
 $Comp
-L ESP8266:ESP8266EX U1
+L WirelessEStop_Tx-rescue:ESP8266EX-ESP8266 U1
 U 1 1 5DE888E0
 P 3650 2750
@@
 Wire Wire Line
 	8450 5400 8450 5300
+NoConn ~ 3700 3550
 $EndSCHEMATC

Commit message: rev 2 work yay
Parts:
- removed C11, C9: .1uF, Capacitor_SMD:C_0603_1608Metric_Pad1.05x0.95mm_HandSolder, symbol Device:C
- removed C3: 3.0pF, Capacitor_SMD:C_0603_1608Metric_Pad1.05x0.95mm_HandSolder, symbol Device:C
- removed C5, C6: 10pF, Capacitor_SMD:C_0603_1608Metric_Pad1.05x0.95mm_HandSolder, symbol Device:C
- removed D9: D, LED_SMD:LED_0603_1608Metric_Pad1.05x0.95mm_HandSolder, symbol Device:D
- removed J1: U.FL-R-SMT(01), U.FL-R-SMT_01_:HRS_U.FL-R-SMT(01), symbol WirelessEStop_Tx-rescue:U.FL-R-SMT(01)-U.FL-R-SMT_01_
- removed L1: 2.2nH, Inductor_SMD:L_0603_1608Metric_Pad1.05x0.95mm_HandSolder, symbol pspice:INDUCTOR
- removed R21: 330, Resistor_SMD:R_0603_1608Metric_Pad1.05x0.95mm_HandSolder, symbol Device:R
- removed R5: 12k, Resistor_SMD:R_0603_1608Metric_Pad1.05x0.95mm_HandSolder, symbol Device:R
- removed R6: 10k, Resistor_SMD:R_0603_1608Metric_Pad1.05x0.95mm_HandSolder, symbol Device:R
- removed R8: 200, Resistor_SMD:R_0603_1608Metric_Pad1.05x0.95mm_HandSolder, symbol Device:R
- removed U1: ESP8266EX, ESP8266:ESP2866EX_Chip, symbol WirelessEStop_Tx-rescue:ESP8266EX-ESP8266
- removed U2: 25Q128FV, W25Q128FVSIF:SOIC127P600X175-8N, symbol WirelessEStop_Tx-rescue:25Q128FV-25Q128FV
- removed Y1: Crystal_GND24, Crystal:Crystal_SMD_2016-4Pin_2.0x1.6mm, symbol Device:Crystal_GND24
- added U1: ESP-13-WROOM-02, ESP8266:MODULE_ESP-WROOM-02U, symbol ESP8266:ESP-13-WROOM-02
- C1: value 2.4pF -> 0.1uF
- C2: value .1uF -> 0.1uF
- J2, J4: footprint Connector_JST:JST_EH_S2B-EH_1x02_P2.50mm_Horizontal -> Connector_JST:JST_EH_B2B-EH-A_1x02_P2.50mm_Vertical
- SW1: footprint Button_Switch_THT:SW_CuK_JS202011AQN_DPDT_Angled -> Connector_JST:JST_EH_B2B-EH-A_1x02_P2.50mm_Vertical
- SW2: footprint Button_Switch_THT:SW_CuK_JS202011CQN_DPDT_Straight -> Connector_JST:JST_EH_B2B-EH-A_1x02_P2.50mm_Vertical
- SW3: footprint Button_Switch_SMD:SW_SPST_TL3305A -> Connector_JST:JST_EH_B2B-EH-A_1x02_P2.50mm_Vertical
- SW6: footprint MRDT_Switches:1P2T_Angled_Slide_GPI-152-3013 -> Connector_JST:JST_EH_B3B-EH-A_1x03_P2.50mm_Vertical
- U4: footprint (none) -> MCP73831T-2ACI_OT:SOT95P280X145-5N
- U5: footprint (none) -> TPS73633DBVR:SOT95P280X145-5N
Connections:
- net +3V3: now also U1.1 (VCC); no longer R23.2
- net ADC_In: now also U1.16 (TOUT)
- net GND: now also C1.1, D11.1 (K), U1.13 (GND), U1.18 (GND), U1.9 (GND), U1.PAD (GND); no longer C1.2
- net I2C_CLK: now also U1.3 (GPIO14)
- net I2C_SDA: now also U1.7 (GPIO2)
- net IND_Connected: now also U1.5 (GPIO13)
- net IND_LowBattery: now also U1.10 (GPIO4)
- net IND_Software: now also R28.2, U1.14 (GPIO5); no longer R11.2
- net RXD: now also U1.12 (TXD)
- net SW_Arm: now also U1.17 (GPIO16)
- net SW_Flash: now also R23.2, U1.6 (GPIO15); no longer D11.1 (K)
- net SW_Reset: now also U1.15 (RST)
- net SW_Trigger: now also U1.4 (GPIO12)
- net TXD: now also R11.2, U1.11 (RXD); no longer R28.2
- net at R1.1: now also C1.2, U1.2 (EN)
- no-connect marks 9 -> 7
Other:
- note removed: "Flash Memory"
- moved on the sheet: C10, R30, R31, U5

Commit message: Finished Rev 2, added silks
Parts:
- SW5: footprint Button_Switch_THT:SW_CuK_JS202011CQN_DPDT_Straight -> Button_Switch_SMD:SW_SPST_TL3305A
Changed lines of the file:
@@
 F 0 "SW5" H 2800 7717 50  0000 C CNN
 F 1 "SW_DIP_x01" H 2800 7626 50  0000 C CNN
-F 2 "Button_Switch_THT:SW_CuK_JS202011CQN_DPDT_Straight" H 2800 7450 50  0001 C CNN
+F 2 "Button_Switch_SMD:SW_SPST_TL3305A" H 2800 7450 50  0001 C CNN
 F 3 "~" H 2800 7450 50  0001 C CNN
 	1    2800 7450

Commit message: Yeet Yeet
Connections:
- net GND: now also U1.6 (GPIO15)
- net SW_Flash: now also U1.8 (GPIO0); no longer U1.6 (GPIO15)
Changed lines of the file:
@@
 Wire Wire Line
 	2450 6750 2500 6750
-Text GLabel 2100 2550 0    39   Output ~ 0
+Text GLabel 2100 2750 0    39   Output ~ 0
 SW_Flash
 Wire Wire Line
@@
 	2150 2450 2100 2450
 Wire Wire Line
-	2100 2550 2150 2550
+	2100 2750 2150 2750
+Wire Wire Line
+	1700 2550 1700 2600
+Wire Wire Line
+	1700 2550 2150 2550
+$Comp
+L power:GND #PWR?
+U 1 1 5E3FECC5
+P 1700 2600
+F 0 "#PWR?" H 1700 2350 50  0001 C CNN
+F 1 "GND" H 1600 2600 50  0000 C CNN
+F 2 "" H 1700 2600 50  0001 C CNN
+F 3 "" H 1700 2600 50  0001 C CNN
+	1    1700 2600
+	1    0    0    -1
+$EndComp
 $EndSCHEMATC

Commit message: Added Documentation
Parts:
- added R5: 0, Resistor_SMD:R_0603_1608Metric_Pad1.05x0.95mm_HandSolder, symbol Device:R
Connections:
- net GND: now also R5.2; no longer U1.6 (GPIO15)
- new net: R5.1, U1.6 (GPIO15)
Changed lines of the file:
@@
 Wire Wire Line
 	2100 2750 2150 2750
-Wire Wire Line
-	1700 2550 1700 2600
-Wire Wire Line
-	1700 2550 2150 2550
 $Comp
-L power:GND #PWR?
+L power:GND #PWR0101
 U 1 1 5E3FECC5
-P 1700 2600
-F 0 "#PWR?" H 1700 2350 50  0001 C CNN
-F 1 "GND" H 1600 2600 50  0000 C CNN
-F 2 "" H 1700 2600 50  0001 C CNN
-F 3 "" H 1700 2600 50  0001 C CNN
-	1    1700 2600
+P 1700 2650
+F 0 "#PWR0101" H 1700 2400 50  0001 C CNN
+F 1 "GND" H 1600 2650 50  0000 C CNN
+F 2 "" H 1700 2650 50  0001 C CNN
+F 3 "" H 1700 2650 50  0001 C CNN
+	1    1700 2650
 	1    0    0    -1
 $EndComp
+$Comp
+L Device:R R5
+U 1 1 5E3D7FB7
+P 1950 2550
+F 0 "R5" V 2000 2400 50  0000 C CNN
+F 1 "0" V 1950 2550 50  0000 C CNN
+F 2 "Resistor_SMD:R_0603_1608Metric_Pad1.05x0.95mm_HandSolder" V 1880 2550 50  0001 C CNN
+F 3 "~" H 1950 2550 50  0001 C CNN
+	1    1950 2550
+	0    1    1    0
+$EndComp
+Wire Wire Line
+	2100 2550 2150 2550
+Wire Wire Line
+	1800 2550 1700 2550
+Wire Wire Line
+	1700 2550 1700 2650
 $EndSCHEMATC
