File: WirelessEStop_Tx.kicad_pcb (KiCad board)
At the start: 2 copper layers, 50.8 x 127 mm, 76 parts, among them IC1 DRV2605LDGSR, J1 U.FL-R-SMT(01), J2 Conn_01x02, J3 USB_B_Micro, J4 Conn_01x02, SW1 SW_Push, SW3 SW_Push, SW4 SW_Push, U1 ESP8266EX, U2 25Q128FV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

Commit message: If you can read this message, please, you need to do something. I'm locked in the github server room, and the things I've seen.... Oh fuck, I think I hear a comp sci coming OH GOD PLEASE NO, HEL......
Parts:
- removed C4: C, Capacitor_SMD:C_0603_1608Metric_Pad1.05x0.95mm_HandSolder
- removed D12, D13: D, LED_SMD:LED_0603_1608Metric_Pad1.05x0.95mm_HandSolder
- removed R24, R25: 330, Resistor_SMD:R_0603_1608Metric_Pad1.05x0.95mm_HandSolder
- added SW2: SW_DIP_x01, Button_Switch_THT:SW_CuK_JS202011CQN_DPDT_Straight, F.Cu at (139.1, 63.6)
- added SW5: SW_DIP_x01, Button_Switch_THT:SW_CuK_JS202011CQN_DPDT_Straight, F.Cu at (104.1, 158.9)
- SW1: value SW_Push -> SW_DIP_x01; footprint Button_Switch_SMD:SW_Push_1P1T_NO_CK_PTS125Sx43PSMTR -> Button_Switch_THT:SW_CuK_JS202011CQN_DPDT_Straight
- SW3, SW4: footprint Button_Switch_SMD:SW_Push_1P1T_NO_CK_PTS125Sx43PSMTR -> Button_Switch_SMD:SW_SPST_TL3305A
- moved SW4 117.8 mm to (112.5, 156.5), turned to 90 degrees
- moved D9 103.4 mm to (150.6, 147.9), turned to 270 degrees
- moved R21 92.8 mm to (148.7, 147.9), turned to 270 degrees
- moved R5 74.0 mm to (122.9, 142.2), turned to 180 degrees
- moved SW1 72.5 mm to (59.0, 127.4)
- moved D11 70.0 mm to (105.9, 150.2), turned to 180 degrees
- moved R23 64.7 mm to (105.9, 148.3)
- moved SW3 63.1 mm to (83.1, 135.4), turned to 270 degrees
- moved R22 60.9 mm to (92.8, 139.8)
- moved IC1 23.3 mm to (160.7, 154.3)
- moved U3 22.8 mm to (149.2, 139.1)
- moved R19 19.5 mm to (94.4, 148.5)
- moved C5 15.0 mm to (126.1, 139.8), turned to 180 degrees
- moved J1 14.4 mm to (116.9, 146.2), turned to 90 degrees
- moved R8 14.2 mm to (133.5, 146.5)
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Connections:
- D11 pad 1: GND -> SW_Flash
- D14 pad 1: GND -> I2C_SDA
- D9 pad 1: GND -> SD_CMD
- R21 pad 2: SW_Reset -> +3V3
- R23 pad 2: SW_Flash -> +3V3
- R26 pad 2: I2C_SDA -> +3V3
- SW1 pad 1: +3V3 -> Net-(SW1-Pad1)
- SW1 pad 2: GND -> Net-(SW1-Pad2)
- U1 pad 29: Net-(C4-Pad2) -> +3V3
- U1 pad 30: Net-(C4-Pad2) -> +3V3
Routing:
- net D-: track 15.3 -> 3.43 mm
- net D+: track 14.4 -> 2.62 mm
- net SW_Flash: track 0.00 -> 9.73 mm
- net SW_Reset: track 0.00 -> 9.07 mm, vias 0 -> 1
- net +3V3: track 19.8 -> 27.7 mm
- net Net-(R5-Pad1): track 0.00 -> 4.12 mm
- net Net-(C6-Pad2): track 11.0 -> 7.94 mm
- net Net-(D9-Pad2): track 0.00 -> 2.55 mm
- net RXD: track 11.9 -> 9.66 mm
- net TXD: track 12.8 -> 10.7 mm
- net Net-(D11-Pad2): track 0.00 -> 1.91 mm
Other:
- board text added: "Battery"
- board text added: "Motor"
- board text added: "RST"

Commit message: big pp
Parts:
- moved SW1 106.0 mm to (121.3, 41.7)
- moved R1 82.5 mm to (120.7, 151.4)
- moved C2 82.1 mm to (120.7, 153.3), turned to 180 degrees
- moved L1 80.6 mm to (121.3, 146.1)
- moved C1 76.2 mm to (121.3, 148.0)
- moved C3 75.9 mm to (121.3, 144.1)
- moved C11 72.0 mm to (117.3, 140.4)
- moved R30 68.5 mm to (141.0, 69.7), turned to 180 degrees
- moved C10 63.9 mm to (117.3, 142.2)
- moved IC1 50.8 mm to (111.3, 142.4), turned to 90 degrees
- moved R31 50.8 mm to (141.0, 72.1)
- moved D9 12.2 mm to (139.5, 142.8), turned to 0 degrees
- moved R21 10.4 mm to (138.6, 145.4)
- moved U3 9.99 mm to (143.5, 147.3), turned to 90 degrees
- moved U2 5.98 mm to (135.0, 147.3), turned to 270 degrees
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Routing:
- net +BATT: track 0.00 -> 41.4 mm
- net SD_D1: track 21.7 -> 4.75 mm
- net SD_D3: track 25.0 -> 10.4 mm, vias 2 -> 0
- net GND: track 10.3 -> 0.97 mm, vias 5 -> 3
- net ADC_VDiv: track 0.00 -> 7.41 mm
- net SD_CMD: track 23.1 -> 15.8 mm, vias 2 -> 0
- net Net-(R30-Pad2): track 0.00 -> 7.24 mm
- net +3V3: track 27.7 -> 33.1 mm
- net D-: track 3.43 -> 0.00 mm
- net SW_Arm: track 0.00 -> 3.36 mm
- net RXD: track 9.66 -> 6.84 mm, vias 0 -> 1
- net D+: track 2.62 -> 0.00 mm
- net SW_Flash: track 9.73 -> 11.6 mm
- net Net-(R8-Pad2): track 3.39 -> 1.52 mm, vias 0 -> 1
- net TXD: track 10.7 -> 9.26 mm, vias 0 -> 1
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Other:
- board text added: "FLSH"
- board text added: "Memory"
- board text added: "OFF"
- board text added: "ON"

Commit message: Eli suck my dick
Parts:
- moved D1 105.7 mm to (146.1, 152.4), turned to 180 degrees
- moved R12 99.0 mm to (150.4, 151.5), turned to 90 degrees
- moved C9 70.9 mm to (112.5, 148.3)
- moved R2 68.6 mm to (121.9, 54.2)
- moved R27 66.8 mm to (95.3, 154.6), turned to 90 degrees
- moved R9 66.2 mm to (110.4, 143.4), turned to 90 degrees
- moved R6 65.3 mm to (112.5, 146.4)
- moved C12 64.6 mm to (103.5, 143.5), turned to 90 degrees
- moved R7 60.9 mm to (108.6, 143.4), turned to 90 degrees
- moved D8 60.8 mm to (104.5, 134.4), turned to 180 degrees
- moved C13 59.6 mm to (103.5, 139.8), turned to 270 degrees
- moved R20 59.0 mm to (104.5, 136.2)
- moved R4 58.5 mm to (128.6, 51.5)
- moved R3 49.8 mm to (123.0, 50.5)
- moved U3 17.6 mm to (127.0, 153.4), turned to 0 degrees
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Connections:
- U1 pad 29: +3V3 -> Net-(C10-Pad2)
- U1 pad 30: +3V3 -> Net-(C10-Pad2)
Routing:
- net Motor-: track 0.00 -> 91.5 mm, vias 0 -> 1
- net Motor+: track 0.00 -> 79.6 mm, vias 0 -> 1
- net Net-(C10-Pad2): track 0.00 -> 25.2 mm, vias 0 -> 3
- net +3V3: track 33.1 -> 49.8 mm
- net Net-(R8-Pad2): track 1.52 -> 17.1 mm, vias 1 -> 2
- net SW_Reset: track 9.07 -> 24.5 mm, vias 1 -> 0
- net SD_D0: track 11.3 -> 25.2 mm
- net SW_Arm: track 3.36 -> 10.6 mm
- net D+: track 0.00 -> 7.09 mm
- net D-: track 0.00 -> 6.09 mm
- net TXD: track 9.26 -> 15.0 mm, vias 1 -> 2
- net SD_D1: track 4.75 -> 9.98 mm
- net Net-(C3-Pad1): track 0.00 -> 4.93 mm
- net Net-(R5-Pad1): track 4.12 -> 8.76 mm
- net I2C_CLK: track 0.00 -> 4.59 mm, vias 0 -> 2
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Other:
- rule trace_min: 0.2 -> 0

Commit message: The only thing longer than my commit names are... MY LOVE OF JESUS CHRIST CAN I GET AN AMEN?
Parts:
- moved R22 99.3 mm to (132.3, 48.7)
- moved D10 98.3 mm to (133.6, 52.0)
- moved D14 92.8 mm to (146.5, 140.8), turned to 180 degrees
- moved D5 84.7 mm to (117.0, 151.0), turned to 180 degrees
- moved R10 80.9 mm to (117.0, 152.8)
- moved R26 80.2 mm to (140.4, 145.5), turned to 270 degrees
- moved C7 77.5 mm to (112.5, 144.5)
- moved D15 69.1 mm to (98.0, 155.1), turned to 90 degrees
- moved D7 66.7 mm to (94.4, 150.6), turned to 180 degrees
- moved R14 64.9 mm to (112.5, 142.6), turned to 180 degrees
- moved R15 63.0 mm to (112.5, 140.7), turned to 180 degrees
- moved D6 33.0 mm to (90.7, 85.8), turned to 180 degrees
- moved R9 4.01 mm to (108.6, 139.8), turned to 270 degrees
- moved C9 1.91 mm to (112.5, 146.4)
- moved R6 1.91 mm to (112.5, 148.3), turned to 180 degrees
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Connections:
- U1 pad 12: IND_Connected -> IND_Software
- U1 pad 8: IND_Software -> IND_Connected
Routing:
- net +3V3: track 49.8 -> 139.9 mm, vias 0 -> 3
- net +BATT: track 41.4 -> 124.4 mm, vias 0 -> 2
- net I2C_SDA: track 2.25 -> 41.3 mm, vias 2 -> 3
- net I2C_CLK: track 4.59 -> 31.8 mm, vias 2 -> 3
- net IND_Connected: track 0.00 -> 13.8 mm, vias 0 -> 2
- net GND: track 4.47 -> 15.9 mm, vias 13 -> 14
- net SW_Reset: track 24.5 -> 30.7 mm
- net Motor-: track 91.5 -> 85.5 mm
- net Motor+: track 79.6 -> 83.9 mm
- net IND_LowBattery: track 3.73 -> 7.92 mm, vias 0 -> 1
- net IND_Software: track 4.34 -> 1.48 mm, vias 0 -> 1
- net IND_Arm: track 0.00 -> 2.50 mm, vias 0 -> 1
- net Net-(D5-Pad2): track 0.00 -> 1.85 mm
- net Net-(D8-Pad2): track 0.00 -> 1.83 mm
- net SW_Trigger: track 2.90 -> 1.70 mm
Other:
- board text added: "Conn"
- board text added: "MMRY"
- board text removed: "Memory"

Commit message: Bout to be date time with the ESP (Extra special person)
Parts:
- moved C2 1.30 mm to (121.3, 151.8), turned to 180 degrees
- moved R1 1.16 mm to (121.3, 149.9), turned to 180 degrees
Routing:
- net GND: track 15.9 -> 22.7 mm, vias 14 -> 15
- net +3V3: track 139.9 -> 135.2 mm
- net +BATT: track 124.4 -> 128.1 mm, vias 2 -> 1
- net Net-(R1-Pad1): track 2.76 -> 0.51 mm

Commit message: Please let the sweet release of death take me soon
Parts:
- added Q1: Q_NMOS_GSD, IRLML6344TRPBF:SOT95P240X112-3N, F.Cu at (129.2, 52.3)
- SW1: footprint Button_Switch_THT:SW_CuK_JS202011CQN_DPDT_Straight -> Button_Switch_THT:SW_CuK_JS202011AQN_DPDT_Angled
- moved D7 115.7 mm to (128.4, 40.0)
- moved R19 115.7 mm to (128.4, 37.9)
- moved D16 100.3 mm to (157.4, 136.4), turned to 180 degrees
- moved R28 87.6 mm to (157.4, 138.2)
- moved R11 87.5 mm to (150.4, 147.8), turned to 270 degrees
- moved D6 83.9 mm to (146.1, 148.7)
- moved SW3 83.7 mm to (106.9, 55.1), turned to 90 degrees
- moved R27 61.4 mm to (156.6, 144.1), turned to 0 degrees
- moved D15 60.0 mm to (156.6, 142.4), turned to 180 degrees
- moved D14 43.8 mm to (104.4, 128.8)
- moved R26 38.9 mm to (104.4, 130.7), turned to 0 degrees
- moved SW1 15.4 mm to (135.3, 48.2), turned to 120 degrees
- moved D10 12.9 mm to (120.8, 50.2)
- moved R22 12.0 mm to (120.8, 52.0), turned to 180 degrees
- moved R2 10.8 mm to (131.7, 49.7), turned to 90 degrees
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Connections:
- R19 pad 2: IND_Arm -> SW_Arm
- SW1 pad 1: Net-(SW1-Pad1) -> +3V3
- SW1 pad 2: Net-(SW1-Pad2) -> SW_Arm
Routing:
- net ADC_VDiv: track 7.41 -> 113.6 mm, vias 0 -> 2
- net +3V3: track 135.2 -> 197.2 mm, vias 3 -> 8
- net IND_LowBattery: track 7.92 -> 39.5 mm, vias 1 -> 2
- net IND_Software: track 1.48 -> 32.4 mm, vias 1 -> 2
- net ADC_In: track 0.87 -> 22.2 mm, vias 1 -> 2
- net SW_Reset: track 30.7 -> 45.6 mm, vias 0 -> 2
- net GND: track 22.7 -> 32.6 mm, vias 15 -> 27
- net Net-(C1-Pad1): track 3.96 -> 10.7 mm
- net Net-(D1-Pad2): track 0.00 -> 6.64 mm
- net Net-(D6-Pad2): track 0.00 -> 6.63 mm
- net SW_Arm: track 10.6 -> 16.3 mm, vias 0 -> 1
- net Net-(R5-Pad1): track 8.76 -> 5.53 mm
- net Net-(R1-Pad1): track 0.51 -> 2.84 mm
- net IND_Connected: track 13.8 -> 12.1 mm
- net I2C_CLK: track 31.8 -> 30.5 mm
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Other:
- board text added: "I2C"
- board text added: "LW BTRY"
- board text added: "Mem"
- board text removed: "MMRY"

Commit message: l
Parts:
- R18: value 2k -> 2k2
- moved D16 12.3 mm to (146.1, 141.4)
- moved D15 10.8 mm to (146.1, 145.0)
- moved R28 7.31 mm to (150.4, 140.5), turned to 90 degrees
- moved R27 6.16 mm to (150.4, 144.1), turned to 90 degrees
Connections:
- C10 pad 2: Net-(C10-Pad2) -> GND
- C11 pad 2: Net-(C10-Pad2) -> GND
- R27 pad 2: TXD -> RXD
- R28 pad 2: RXD -> TXD
- U1 pad 1: Net-(C10-Pad2) -> +3V3
- U1 pad 25: RXD -> TXD
- U1 pad 26: TXD -> RXD
- U1 pad 29: Net-(C10-Pad2) -> +3V3
- U1 pad 3: Net-(C10-Pad2) -> +3V3
- U1 pad 30: Net-(C10-Pad2) -> +3V3
- U1 pad 4: Net-(C10-Pad2) -> +3V3
Routing:
- net SW_Arm: track 16.3 -> 116.8 mm
- net +3V3: track 197.2 -> 227.9 mm, vias 8 -> 11
- net RXD: track 11.3 -> 39.0 mm, vias 2 -> 3
- net TXD: track 15.0 -> 41.0 mm, vias 2 -> 3
- net Net-(C10-Pad2): track 24.3 -> 0.00 mm, vias 3 -> 0
- net I2C_SDA: track 41.8 -> 54.5 mm
- net Net-(D16-Pad2): track 0.00 -> 7.54 mm
- net Net-(D15-Pad2): track 0.00 -> 6.53 mm
- net SD_D1: track 9.98 -> 13.6 mm
- net Net-(D14-Pad2): track 0.00 -> 1.85 mm
- net +BATT: track 128.3 -> 127.6 mm
- net GND: vias 27 -> 38
Other:
- board text added: "MMRY"
- board text added: "RX"
- board text added: "Software"
- board text added: "TX"
- board text removed: "Mem"

Commit message: Rethinkimg things
Parts:
- moved SW1 8.12 mm to (141.6, 53.3)
- moved R30 5.46 mm to (146.4, 69.7)
- moved R31 5.46 mm to (146.4, 72.1)
- moved SW2 5.46 mm to (142.6, 63.5)
- moved U5 5.46 mm to (146.4, 66.0)
- moved J4 5.46 mm to (121.0, 68.7)
- moved J2 5.46 mm to (133.7, 63.5)
- moved C5 0.38 mm to (126.1, 139.4)
- moved C6 0.38 mm to (129.8, 139.4)
Routing:
- net Motor-: track 85.5 -> 14.1 mm
- net ADC_VDiv: track 113.6 -> 143.9 mm
- net SW_Flash: track 13.2 -> 39.2 mm, vias 1 -> 3
- net Motor+: track 83.9 -> 107.9 mm
- net SW_Trigger: track 1.70 -> 17.2 mm, vias 1 -> 2
- net +3V3: track 227.9 -> 238.3 mm
- net SW_Arm: track 116.8 -> 106.9 mm
- net +BATT: track 127.6 -> 118.0 mm
- net IND_Arm: track 2.50 -> 0.01 mm, vias 1 -> 0
- net GND: track 32.6 -> 35.1 mm, vias 38 -> 35
- net Net-(R8-Pad2): track 17.1 -> 19.1 mm
- net Net-(C6-Pad2): track 7.94 -> 9.70 mm
- net Net-(C5-Pad2): track 6.17 -> 7.12 mm
- net SW_Reset: track 45.6 -> 44.6 mm
Other:
- outline, holes or cut-outs redrawn
