File: WirelessEStop_Tx.kicad_pcb (KiCad board)
At the start: 2 copper layers, 50.8 x 127 mm, 74 parts, among them IC1 DRV2605LDGSR, J1 U.FL-R-SMT(01), J2 Conn_01x02, J3 USB_B_Micro, J4 Conn_01x02, Q1 Q_NMOS_GSD, SW1 SW_DIP_x01, SW2 SW_DIP_x01, SW3 SW_Push, SW4 SW_Push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

Commit message: Whats the difference between Dahlbot, and a baby? I dont want to strangle Dahlbot to death
Parts:
- added ?: , , F.Cu at (104.4, 132.5)
- added SW6: SW_SPDT, Connector_JST:JST_EH_B3B-EH-A_1x03_P2.50mm_Vertical, F.Cu at (118.7, 122.5)
- J2, J4: footprint Connector_JST:JST_EH_S2B-EH_1x02_P2.50mm_Horizontal -> Connector_JST:JST_EH_B2B-EH-A_1x02_P2.50mm_Vertical
- SW1: footprint Button_Switch_THT:SW_CuK_JS202011AQN_DPDT_Angled -> Connector_JST:JST_EH_B2B-EH-A_1x02_P2.50mm_Vertical
- SW2: footprint Button_Switch_THT:SW_CuK_JS202011CQN_DPDT_Straight -> Connector_JST:JST_EH_B2B-EH-A_1x02_P2.50mm_Vertical
- SW3: footprint Button_Switch_SMD:SW_SPST_TL3305A -> Connector_JST:JST_EH_B2B-EH-A_1x02_P2.50mm_Vertical
- moved D7 95.4 mm to (139.3, 134.7)
- moved R19 95.4 mm to (139.3, 132.7)
- moved R2 82.1 mm to (116.6, 130.4), turned to 180 degrees
- moved D10 78.6 mm to (125.3, 128.7), turned to 180 degrees
- moved R4 77.5 mm to (116.7, 126.7), turned to 180 degrees
- moved Q1 75.8 mm to (121.0, 127.7), turned to 0 degrees
- moved R3 75.8 mm to (116.7, 128.6), turned to 180 degrees
- moved SW1 75.5 mm to (145.2, 128.8), turned to 0 degrees
- moved R22 75.0 mm to (125.3, 126.9), turned to 0 degrees
- moved SW3 67.4 mm to (106.3, 122.5), turned to 0 degrees
- moved U5 63.3 mm to (132.6, 127.8), turned to 0 degrees
- moved J4 61.8 mm to (106.3, 128.8)
- moved J2 60.0 mm to (145.2, 122.4), turned to 0 degrees
- moved SW2 59.7 mm to (133.3, 122.4), turned to 0 degrees
- moved R30 59.0 mm to (135.9, 127.8), turned to 270 degrees
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Connections:
- net IND_Arm renamed Net-(U1-Pad13)
Routing:
- net ADC_VDiv: track 143.9 -> 9.56 mm, vias 2 -> 1
- net Motor+: track 107.9 -> 12.9 mm
- net SW_Arm: track 106.9 -> 30.0 mm
- net +BATT: track 118.0 -> 54.5 mm
- net +3V3: track 238.3 -> 197.9 mm
- net Net-(R3-Pad2): track 0.00 -> 19.8 mm
- net Net-(Q1-Pad3): track 0.00 -> 15.0 mm
- net SW_Trigger: track 17.2 -> 30.6 mm
- net GND: track 35.1 -> 43.9 mm, vias 35 -> 42
- net Net-(R30-Pad2): track 7.24 -> 0.00 mm
- net Motor-: track 14.1 -> 19.5 mm
- net DC_In: track 24.8 -> 29.3 mm
- net ADC_In: track 22.2 -> 25.9 mm
- net I2C_SDA: track 54.9 -> 51.5 mm, vias 4 -> 5
- net D-: track 6.09 -> 9.47 mm
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Other:
- board size 50.8 x 127 mm -> 50.8 x 47.8 mm
- board text added: "+"
- board text added: "-"
- board text added: "Motor Port"
- board text added: "TRGR"
- board text added: "Trigger Port"
- board text removed: "Battery"
- board text removed: "OFF"
- board text removed: "ON"

Commit message: IDK dude, just think of a clever joke and give me credit for it. I just want to play dota
Parts:
- moved D7 4.07 mm to (143.4, 134.8)
- moved R19 4.07 mm to (143.4, 132.8)
Routing:
- net ADC_VDiv: track 9.56 -> 45.2 mm
- net +3V3: track 197.9 -> 216.2 mm
- net SW_Trigger: track 30.6 -> 48.2 mm, vias 2 -> 3
- net SW_Arm: track 30.0 -> 35.4 mm
- net Net-(R30-Pad2): track 0.00 -> 4.06 mm
- net GND: track 43.9 -> 46.9 mm
- net Net-(D7-Pad2): track 0.00 -> 2.03 mm
Other:
- outline, holes or cut-outs redrawn
- board text added: "Toggle Trigger"

Commit message: I ate myself anf was dissapointed
Other:
- outline, holes or cut-outs redrawn
- board text added: "ARM"
- board text added: "Arm Port"
- board text added: "Battery Port"
- board text added: "On/Off Port"
- board text added: "S"
- board text added: "Toggle Port"
- board text added: "Wireless E-Stop Rev 1 Mars Rover Design Team Missouri S&T, 2020 Dan Napierkowski"
- board text removed: "Toggle Trigger"
Changed lines of the file:
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@@
   (general
     (thickness 1.6)
-    (drawings 45)
+    (drawings 61)
     (tracks 872)
     (zones 0)
@@
     (at 132.588 127.762)
     (attr smd)
-    (fp_text reference U5 (at 0 -0.127 270) (layer B.SilkS)
+    (fp_text reference U5 (at -0.889 -0.127) (layer B.SilkS)
       (effects (font (size 1.64087 1.64087) (thickness 0.05)) (justify mirror))
     )
@@
     (tags "resistor handsolder")
     (attr smd)
-    (fp_text reference R31 (at 0 0.0635 90) (layer B.SilkS)
+    (fp_text reference R31 (at 0.014 0.635 180) (layer B.SilkS)
       (effects (font (size 1 1) (thickness 0.15)) (justify mirror))
     )
@@
     (tags "resistor handsolder")
     (attr smd)
-    (fp_text reference R30 (at 0 -0.0635 90) (layer B.SilkS)
+    (fp_text reference R30 (at 0 0.635 180) (layer B.SilkS)
       (effects (font (size 1 1) (thickness 0.15)) (justify mirror))
     )
@@
     (tags "resistor handsolder")
     (attr smd)
-    (fp_text reference R28 (at 0 0.029 90) (layer B.SilkS)
+    (fp_text reference R28 (at -1.016 -0.0635 180) (layer B.SilkS)
       (effects (font (size 1 1) (thickness 0.15)) (justify mirror))
     )
@@
     (tags "resistor handsolder")
     (attr smd)
-    (fp_text reference R19 (at 0 0) (layer B.SilkS)
+    (fp_text reference R19 (at 2.9337 0) (layer B.SilkS)
       (effects (font (size 1 1) (thickness 0.15)) (justify mirror))
     )
@@
     (tags "LED handsolder")
     (attr smd)
-    (fp_text reference D16 (at -0.0495 0) (layer B.SilkS)
+    (fp_text reference D16 (at -0.8255 -0.127) (layer B.SilkS)
       (effects (font (size 1 1) (thickness 0.15)) (justify mirror))
     )
@@
     (tags "LED handsolder")
     (attr smd)
-    (fp_text reference D7 (at 0 0) (layer B.SilkS)
+    (fp_text reference D7 (at -2.9337 -0.0381) (layer B.SilkS)
       (effects (font (size 1 1) (thickness 0.15)) (justify mirror))
     )
@@
     )
   )
-  (gr_text "Toggle Trigger" (at 121.2215 119.634) (layer F.SilkS)
+  (gr_text "On/Off Port" (at 134.5565 119.761) (layer F.SilkS)
+    (effects (font (size 1 1) (thickness 0.25)))
+  )
+  (gr_text "Battery Port" (at 146.3675 119.634) (layer F.SilkS)
+    (effects (font (size 1 1) (thickness 0.25)))
+  )
+  (gr_text "Arm Port" (at 146.3675 125.984) (layer F.SilkS)
+    (effects (font (size 1 1) (thickness 0.25)))
+  )
+  (gr_text - (at 147.5105 130.81) (layer B.SilkS)
+    (effects (font (size 1 1) (thickness 0.25)) (justify mirror))
+  )
+  (gr_text + (at 145.0975 130.81) (layer B.SilkS)
+    (effects (font (size 1 1) (thickness 0.25)) (justify mirror))
+  )
+  (gr_text - (at 145.2245 124.46) (layer B.SilkS)
+    (effects (font (size 1 1) (thickness 0.25)) (justify mirror))
+  )
+  (gr_text + (at 147.6375 124.46) (layer B.SilkS)
+    (effects (font (size 1 1) (thickness 0.25)) (justify mirror))
+  )
+  (gr_text - (at 135.9535 124.46) (layer B.SilkS)
+    (effects (font (size 1 1) (thickness 0.25)) (justify mirror))
+  )
+  (gr_text + (at 133.2865 124.46) (layer B.SilkS)
+    (effects (font (size 1 1) (thickness 0.25)) (justify mirror))
+  )
+  (gr_text S (at 121.2215 124.587) (layer B.SilkS)
+    (effects (font (size 1 1) (thickness 0.25)) (justify mirror))
+  )
+  (gr_text S (at 123.7615 124.587) (layer B.SilkS)
+    (effects (font (size 1 1) (thickness 0.25)) (justify mirror))
+  )
+  (gr_text S (at 118.5545 124.587) (layer B.SilkS)
+    (effects (font (size 1 1) (thickness 0.25)) (justify mirror))
+  )
+  (gr_text S (at 106.2355 124.587) (layer B.SilkS)
+    (effects (font (size 1 1) (thickness 0.25)) (justify mirror))
+  )
+  (gr_text + (at 108.7755 124.46) (layer B.SilkS)
+    (effects (font (size 1 1) (thickness 0.25)) (justify mirror))
+  )
+  (gr_text ARM (at 143.51 136.652) (layer F.SilkS)
+    (effects (font (size 1 1) (thickness 0.25)))
+  )
+  (gr_text "Wireless E-Stop Rev 1\nMars Rover Design Team\nMissouri S&T, 2020\nDan Napierkowski" (at 132.334 133.604) (layer B.SilkS)
+    (effects (font (size 1 1) (thickness 0.25)) (justify mirror))
+  )
+  (gr_text "Toggle Port" (at 121.2215 119.634) (layer F.SilkS)
     (effects (font (size 1 1) (thickness 0.25)))
   )
@@
   (gr_line (start 102.616 118.11) (end 151.384 118.11) (layer Edge.Cuts) (width 0.1))
   (gr_circle (center 150.1775 160.3175) (end 151.4275 160.3175) (layer Edge.Cuts) (width 0.1))
-  (gr_circle (center 134.112 138.938) (end 135.302625 138.938) (layer Edge.Cuts) (width 0.1))
-  (gr_text RX (at 146.1135 139.446) (layer F.SilkS)
+  (gr_circle (center 118.491 134.493) (end 119.681625 134.493) (layer Edge.Cuts) (width 0.1))
+  (gr_text RX (at 146.1135 143.256) (layer F.SilkS)
     (effects (font (size 1 1) (thickness 0.25)))
   )
-  (gr_text TX (at 146.1135 143.256) (layer F.SilkS)
+  (gr_text TX (at 146.177 139.446) (layer F.SilkS)
     (effects (font (size 1 1) (thickness 0.25)))
   )

Commit message: Zak your name is weird since its only 3 letters, but its also as many letters as needed. Its a weird juxtaposition of right and wrong and it makes me uncomfortable
Parts:
- added G***: LOGO, ESP8266:Signature, B.Cu at (139.8, 160.4)
- added G***: LOGO, ESP8266:lizard_logo, B.Cu at (133.3, 133.5)
