File: WirelessEStop_Tx.kicad_pcb (KiCad board)
At the start: 2 copper layers, 50.8 x 47.8 mm, 78 parts, among them IC1 DRV2605LDGSR, J1 U.FL-R-SMT(01), J2 Conn_01x02, J3 USB_B_Micro, J4 Conn_01x02, Q1 Q_NMOS_GSD, SW1 SW_DIP_x01, SW2 SW_DIP_x01, SW3 SW_Push, SW4 SW_Push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

Commit message: rev 2 work yay
Parts:
- removed ?: , 
- removed C11, C9: .1uF, Capacitor_SMD:C_0603_1608Metric_Pad1.05x0.95mm_HandSolder
- removed C3: 3.0pF, Capacitor_SMD:C_0603_1608Metric_Pad1.05x0.95mm_HandSolder
- removed C5, C6: 10pF, Capacitor_SMD:C_0603_1608Metric_Pad1.05x0.95mm_HandSolder
- removed D9: D, LED_SMD:LED_0603_1608Metric_Pad1.05x0.95mm_HandSolder
- removed G***: LOGO, ESP8266:Signature
- removed G***: LOGO, ESP8266:lizard_logo
- removed J1: U.FL-R-SMT(01), U.FL-R-SMT_01_:HRS_U.FL-R-SMT(01)
- removed L1: 2.2nH, Inductor_SMD:L_0603_1608Metric_Pad1.05x0.95mm_HandSolder
- removed R21: 330, Resistor_SMD:R_0603_1608Metric_Pad1.05x0.95mm_HandSolder
- removed R5: 12k, Resistor_SMD:R_0603_1608Metric_Pad1.05x0.95mm_HandSolder
- removed R6: 10k, Resistor_SMD:R_0603_1608Metric_Pad1.05x0.95mm_HandSolder
- removed R8: 200, Resistor_SMD:R_0603_1608Metric_Pad1.05x0.95mm_HandSolder
- removed U2: 25Q128FV, W25Q128FVSIF:SOIC127P600X175-8N
- removed Y1: Crystal_GND24, Crystal:Crystal_SMD_2016-4Pin_2.0x1.6mm
- C1: value 2.4pF -> 0.1uF
- C2: value .1uF -> 0.1uF
- SW5: footprint Button_Switch_THT:SW_CuK_JS202011CQN_DPDT_Straight -> Button_Switch_SMD:SW_SPST_TL3305A
- U1: value ESP8266EX -> ESP-13-WROOM-02; footprint ESP8266:ESP2866EX_Chip -> ESP8266:MODULE_ESP-WROOM-02U
- U5: footprint MCP73831T-2ACI_OT:SOT95P280X145-5N -> TPS73633DBVR:SOT95P280X145-5N
- moved R15 29.8 mm to (139.8, 129.0), turned to 90 degrees
- moved R14 29.0 mm to (138.0, 129.0), turned to 90 degrees
- moved C7 28.4 mm to (136.3, 129.0), turned to 270 degrees
- moved R22 20.6 mm to (118.3, 146.2), turned to 180 degrees
- moved C2 19.1 mm to (115.8, 133.5), turned to 180 degrees
- moved D10 17.3 mm to (118.3, 144.5), turned to 0 degrees
- moved R1 13.9 mm to (115.8, 137.2), turned to 0 degrees
- moved C1 10.6 mm to (115.8, 139.1)
- moved U1 8.41 mm to (131.1, 140.0)
- moved R19 8.10 mm to (150.4, 136.8), turned to 90 degrees
- moved D5 7.63 mm to (113.1, 144.5)
- moved R10 7.63 mm to (113.1, 146.3)
- moved C10 6.34 mm to (115.8, 135.4), turned to 180 degrees
- moved U5 5.11 mm to (127.6, 129.0)
- moved D7 3.81 mm to (146.1, 137.5)
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Connections:
- C1 pad 1: Net-(C1-Pad1) -> GND
- C1 pad 2: GND -> Net-(C1-Pad2)
- D11 pad 1: SW_Flash -> GND
- R1 pad 1: Net-(R1-Pad1) -> Net-(C1-Pad2)
- R11 pad 2: IND_Software -> TXD
- R23 pad 2: +3V3 -> SW_Flash
- R28 pad 2: TXD -> IND_Software
- U1 pad 11: +3V3 -> TXD
- U1 pad 12: IND_Software -> RXD
- U1 pad 13: Net-(U1-Pad13) -> GND
- U1 pad 14: I2C_SDA -> IND_Software
- U1 pad 15: SW_Flash -> SW_Reset
- U1 pad 16: SW_Trigger -> ADC_In
- U1 pad 17: +3V3 -> SW_Arm
- U1 pad 18: SD_D2 -> GND
- U1 pad 19: SD_D3 -> (no net)
- U1 pad 2: Net-(C3-Pad1) -> Net-(C1-Pad2)
- U1 pad 3: +3V3 -> I2C_CLK
- U1 pad 4: +3V3 -> SW_Trigger
- U1 pad 5: Net-(U1-Pad5) -> IND_Connected
- U1 pad 6: ADC_In -> SW_Flash
- U1 pad 7: Net-(R1-Pad1) -> I2C_SDA
- U1 pad 8: IND_Connected -> Net-(U1-Pad8)
- U1 pad 9: I2C_CLK -> GND
Routing:
- net +3V3: track 216.2 -> 124.6 mm, vias 11 -> 4
- net SW_Trigger: track 48.2 -> 6.79 mm, vias 3 -> 0
- net SW_Flash: track 39.2 -> 0.43 mm, vias 3 -> 0
- net IND_LowBattery: track 39.5 -> 5.59 mm, vias 2 -> 1
- net IND_Software: track 32.4 -> 5.86 mm, vias 2 -> 0
- net SD_D0: track 25.2 -> 0.00 mm, vias 2 -> 0
- net GND: track 46.9 -> 24.0 mm, vias 42 -> 14
- net I2C_SDA: track 51.5 -> 30.4 mm, vias 5 -> 4
- net TXD: track 41.0 -> 20.5 mm, vias 3 -> 2
- net ADC_VDiv: track 45.2 -> 25.9 mm, vias 1 -> 0
- net SW_Reset: track 44.6 -> 25.5 mm, vias 2 -> 1
- net Net-(R8-Pad2): track 19.1 -> 0.00 mm, vias 2 -> 0
- net RXD: track 39.0 -> 21.4 mm, vias 3 -> 0
- net I2C_CLK: track 30.5 -> 14.7 mm, vias 3 -> 2
- net SD_CMD: track 15.8 -> 0.00 mm
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Other:
- board size 50.8 x 47.8 mm -> 70.4 x 47.8 mm
- board text added: "Wireless E-Stop Rev 2 Mars Rover Design Team Missouri S&T, 2020 Dan Napierkowski"
- board text removed: "MMRY"
- board text removed: "Wireless E-Stop Rev 1 Mars Rover Design Team Missouri S&T, 2020 Dan Napierkowski"

Commit message: Finished Rev 2, added silks
Parts:
- added G***: LOGO, ESP8266:Signature, B.Cu at (127.6, 149.0)
- added G***: LOGO, ESP8266:lizard_logo, B.Cu at (131.0, 141.5)
- moved R23 10.6 mm to (114.6, 152.6), turned to 180 degrees
- moved D11 8.97 mm to (114.6, 150.7)
- moved SW5 5.66 mm to (107.8, 151.6), turned to 0 degrees
- moved D10 5.28 mm to (113.0, 144.8)
- moved R22 5.28 mm to (113.0, 146.6)
- moved SW4 5.08 mm to (107.7, 158.6), turned to 0 degrees
- moved D5 4.52 mm to (117.6, 144.8), turned to 0 degrees
- moved R10 4.52 mm to (117.6, 146.6), turned to 180 degrees
- moved R7 3.75 mm to (108.6, 139.7)
- moved R9 3.72 mm to (108.6, 143.5), turned to 90 degrees
- moved D17 0.76 mm to (116.4, 158.9)
- moved R29 0.76 mm to (116.4, 157.0)
- turned C7 to 90 degrees
Routing:
- net +3V3: track 124.6 -> 188.7 mm, vias 4 -> 5
- net SW_Trigger: track 6.79 -> 42.6 mm, vias 0 -> 2
- net SW_Flash: track 0.43 -> 34.3 mm, vias 0 -> 2
- net SW_Reset: track 25.5 -> 57.2 mm, vias 1 -> 2
- net TXD: track 20.5 -> 38.9 mm
- net I2C_CLK: track 14.7 -> 30.0 mm
- net RXD: track 21.4 -> 35.2 mm, vias 0 -> 2
- net IND_LowBattery: track 5.59 -> 18.8 mm, vias 1 -> 0
- net IND_Connected: track 1.23 -> 13.4 mm
- net I2C_SDA: track 30.4 -> 41.0 mm
- net IND_Software: track 5.86 -> 10.7 mm
- net Net-(D11-Pad2): track 5.38 -> 1.91 mm, vias 1 -> 0
- net GND: track 24.0 -> 27.3 mm, vias 14 -> 20
- net Net-(D10-Pad2): track 0.00 -> 1.78 mm
- net Net-(D5-Pad2): track 0.00 -> 1.78 mm
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Other:
- board size 70.4 x 47.8 mm -> 50.8 x 47.8 mm

Commit message: Yeet Yeet
Parts:
- removed G***: LOGO, ESP8266:Signature
- removed G***: LOGO, ESP8266:lizard_logo
Connections:
- U1 pad 6: SW_Flash -> GND
- U1 pad 8: Net-(U1-Pad8) -> SW_Flash
Routing:
- net SW_Flash: track 34.3 -> 27.5 mm
- net GND: track 27.3 -> 30.8 mm, vias 20 -> 21

Commit message: Whoop Whoop, Zoop Zoop
Parts:
- added G***: LOGO, ESP8266:Signature, B.Cu at (128.1, 148.4)
- added G***: LOGO, ESP8266:lizard_logo, B.Cu at (130.8, 141.2)
- added R5: 0, Resistor_SMD:R_0603_1608Metric_Pad1.05x0.95mm_HandSolder, B.Cu at (115.2, 141.9)
- moved D5 0.07 mm to (117.6, 144.8), turned to 180 degrees
- turned D10 to 180 degrees
Connections:
- U1 pad 6: GND -> Net-(R5-Pad1)
Routing:
- net Net-(R5-Pad1): track 0.00 -> 7.45 mm, vias 0 -> 1
- net GND: track 30.8 -> 29.1 mm
- net Net-(D10-Pad2): track 1.78 -> 2.50 mm
- net Net-(D5-Pad2): track 1.78 -> 2.48 mm
- net SW_Trigger: track 42.6 -> 42.0 mm
Other:
- outline, holes or cut-outs redrawn
